File: Midi Bass Sch/Master Sch.kicad_sch (KiCad schematic)
At the start: 9 parts

Commit message: updated schematic to include solenoids for pluck slave
Parts:
- gave numbers to parts that had none: 9
Changed lines of the file:
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@@
 		(dnp no)
 		(fields_autoplaced yes)
-		(property "Reference" "D?"
+		(property "Reference" "D2"
 			(at 99.06 105.7274 90)
 			(effects
@@
 			(project "Midi Bass Sch"
 				(path "/06818073-fb22-48ee-acc5-6dedd827034e/0dc3b915-e001-48bd-b9bb-7010249087fd"
-					(reference "D?")
+					(reference "D2")
 					(unit 1)
 				)
@@
 		(dnp no)
 		(fields_autoplaced yes)
-		(property "Reference" "D?"
+		(property "Reference" "D1"
 			(at 96.52 40.64 90)
 			(effects
@@
 			(project "Midi Bass Sch"
 				(path "/06818073-fb22-48ee-acc5-6dedd827034e/0dc3b915-e001-48bd-b9bb-7010249087fd"
-					(reference "D?")
+					(reference "D1")
 					(unit 1)
 				)
@@
 		(dnp no)
 		(fields_autoplaced yes)
-		(property "Reference" "R?"
+		(property "Reference" "R5"
 			(at 205.74 63.4999 90)
 			(effects
@@
 			(project "Midi Bass Sch"
 				(path "/06818073-fb22-48ee-acc5-6dedd827034e/0dc3b915-e001-48bd-b9bb-7010249087fd"
-					(reference "R?")
+					(reference "R5")
 					(unit 1)
 				)
@@
 		(dnp no)
 		(fields_autoplaced yes)
-		(property "Reference" "C?"
+		(property "Reference" "C1"
 			(at 86.36 50.1649 0)
 			(effects
@@
 			(project "Midi Bass Sch"
 				(path "/06818073-fb22-48ee-acc5-6dedd827034e/0dc3b915-e001-48bd-b9bb-7010249087fd"
-					(reference "C?")
+					(reference "C1")
 					(unit 1)
 				)
@@
 		(dnp no)
 		(fields_autoplaced yes)
-		(property "Reference" "U?"
+		(property "Reference" "U1"
 			(at 149.5141 38.1 0)
 			(effects
@@
 			(project "Midi Bass Sch"
 				(path "/06818073-fb22-48ee-acc5-6dedd827034e/0dc3b915-e001-48bd-b9bb-7010249087fd"
-					(reference "U?")
+					(reference "U1")
 					(unit 1)
 				)
@@
 		(dnp no)
 		(fields_autoplaced yes)
-		(property "Reference" "R?"
+		(property "Reference" "R3"
 			(at 97.79 96.5199 90)
 			(effects
@@
 			(project "Midi Bass Sch"
 				(path "/06818073-fb22-48ee-acc5-6dedd827034e/0dc3b915-e001-48bd-b9bb-7010249087fd"
-					(reference "R?")
+					(reference "R3")
 					(unit 1)
 				)
@@
 		(dnp no)
 		(fields_autoplaced yes)
-		(property "Reference" "R?"
+		(property "Reference" "R2"
 			(at 86.36 39.3699 90)
 			(effects
@@
 			(project "Midi Bass Sch"
 				(path "/06818073-fb22-48ee-acc5-6dedd827034e/0dc3b915-e001-48bd-b9bb-7010249087fd"
-					(reference "R?")
+					(reference "R2")
 					(unit 1)
 				)
@@
 		(dnp no)
 		(fields_autoplaced yes)
-		(property "Reference" "J?"
+		(property "Reference" "J1"
 			(at 69.8501 123.19 0)
 			(effects
@@
 			(project "Midi Bass Sch"
 				(path "/06818073-fb22-48ee-acc5-6dedd827034e/0dc3b915-e001-48bd-b9bb-7010249087fd"
-					(reference "J?")
+					(reference "J1")
 					(unit 1)
 				)
@@
 		(dnp no)
 		(fields_autoplaced yes)
-		(property "Reference" "R?"
+		(property "Reference" "R4"
 			(at 190.5 64.7699 90)
 			(effects
@@
 			(project "Midi Bass Sch"
 				(path "/06818073-fb22-48ee-acc5-6dedd827034e/0dc3b915-e001-48bd-b9bb-7010249087fd"
-					(reference "R?")
-					(unit 1)
-				)
+					(reference "R4")
+					(unit 1)
+				)

Commit message: updated schematic to include test points for pics
Parts:
- added TP1: MidiIN, symbol Connector:TestPoint
- added TP2: CLKOUT0, symbol Connector:TestPoint
- added TP3: SCL, symbol Connector:TestPoint
- added TP4: SDA, symbol Connector:TestPoint
Connections:
- net I2Cclk: now also TP3.1
- net I2Cdat: now also TP4.1
- net at D2.1 (K), J1.5: now also TP1.1
- no-connect marks 23 -> 22
Other:
- moved on the sheet: R5
