File: Midi Bass Sch/ASolenoidA.kicad_sch (KiCad schematic)
At the start: 105 parts, among them Q29 BDW93C, Q30 BDW93C, Q31 BDW93C, Q32 BDW93C, Q33 BDW93C, Q34 BDW93C, Q35 BDW93C, Q36 BDW93C, Q37 BDW93C, Q38 BDW93C, Q39 BDW93C, Q40 BDW93C, Q41 BDW93C, Q42 BDW93C, Q43 BDW93C, Q44 BDW93C, Q45 BDW93C, Q46 BDW93C, Q47 BDW93C, Q48 BDW93C, U14 LTV-247, U15 LTV-247, U16 LTV-247, U17 LTV-247, U18 LTV-247

Commit message: added footprints to kicad schematic still need footprint for din connector
Parts:
- Q29, Q30, Q31, Q32, Q33, Q34, Q35, Q36, Q37, Q38, Q39, Q40, Q41, Q42, Q43, Q44, Q45, Q46, Q47, Q48: footprint (none) -> Package_TO_SOT_THT:TO-220-3_Vertical
- R118, R119, R120, R121, R122, R123, R124, R125, R126, R127, R128, R129, R130, R131, R132, R133, R134, R135, R136, R137, R138, R139, R140, R141, R142, R143, R144, R145, R146, R147, R148, R149, R150, R151, R152, R153, R154, R155, R156, R157, R158, R159, R160, R161, R162, R163, R164, R165, R166, R167, R168, R169, R170, R171, R172, R173, R174, R175, R176, R177: footprint (none) -> Resistor_SMD:R_0805_2012Metric_Pad1.20x1.40mm_HandSolder

Commit message: working on troubleshooting section of report
Parts:
- renumbered L29 to L33, L30 to L34, L31 to L35, L32 to L36, L33 to L37, L34 to L38, L35 to L39, L36 to L40, L37 to L41, L38 to L42, L39 to L43, L40 to L44, L41 to L45, L42 to L46, L43 to L47, L44 to L48, L45 to L49, L46 to L50, L47 to L51, L48 to L52, Q29 to Q33, Q30 to Q34, Q31 to Q35, Q32 to Q36, Q33 to Q37, Q34 to Q38, Q35 to Q39, Q36 to Q40, Q37 to Q41, Q38 to Q42, Q39 to Q43, Q40 to Q44, Q41 to Q45, Q42 to Q46, Q43 to Q47, Q44 to Q48, Q45 to Q49, Q46 to Q50, Q47 to Q51, Q48 to Q52, R118 to R130, R119 to R131, R120 to R132, R121 to R133, R122 to R134, R123 to R135, R124 to R136, R125 to R137, R126 to R138, R127 to R139, R128 to R140, R129 to R141, R130 to R142, R131 to R143, R132 to R144, R133 to R145, R134 to R146, R135 to R147, R136 to R148, R137 to R149, R138 to R150, R139 to R151, R140 to R152, R141 to R153, R142 to R154, R143 to R155, R144 to R156, R145 to R157, R146 to R158, R147 to R159, R148 to R160, R149 to R161, R150 to R162, R151 to R163, R152 to R164, R153 to R165, R154 to R166, R155 to R167, R156 to R168, R157 to R169, R158 to R170, R159 to R171, R160 to R172, R161 to R173, R162 to R174, R163 to R175, R164 to R176, R165 to R177, R166 to R178, R167 to R179, R168 to R180, R169 to R181, R170 to R182, R171 to R183, R172 to R184, R173 to R185, R174 to R186, R175 to R187, R176 to R188, R177 to R189, U14 to U16, U15 to U17, U16 to U18, U17 to U19, U18 to U20

Commit message: changed transistor for schematic
Parts:
- Q33, Q34, Q35, Q36, Q37, Q38, Q39, Q40, Q41, Q42, Q43, Q44, Q45, Q46, Q47, Q48, Q49, Q50, Q51, Q52: value BDW93C -> STN851-A
Changed lines of the file:
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@@
 			)
 		)
-		(property "Value" "BDW93C"
+		(property "Value" "STN851-A"
 			(at 173.99 67.3099 0)
 			(effects
@@
 			)
 		)
-		(property "Value" "BDW93C"
+		(property "Value" "STN851-A"
 			(at 173.99 97.7899 0)
 			(effects
@@
 			)
 		)
-		(property "Value" "BDW93C"
+		(property "Value" "STN851-A"
 			(at 66.04 34.2899 0)
 			(effects
@@
 			)
 		)
-		(property "Value" "BDW93C"
+		(property "Value" "STN851-A"
 			(at 238.76 132.0799 0)
 			(effects
@@
 			)
 		)
-		(property "Value" "BDW93C"
+		(property "Value" "STN851-A"
 			(at 120.65 34.2899 0)
 			(effects
@@
 			)
 		)
-		(property "Value" "BDW93C"
+		(property "Value" "STN851-A"
 			(at 173.99 130.8099 0)
 			(effects
@@
 			)
 		)
-		(property "Value" "BDW93C"
+		(property "Value" "STN851-A"
 			(at 173.99 35.5599 0)
 			(effects
@@
 			)
 		)
-		(property "Value" "BDW93C"
+		(property "Value" "STN851-A"
 			(at 63.5 99.0599 0)
 			(effects
@@
 			)
 		)
-		(property "Value" "BDW93C"
+		(property "Value" "STN851-A"
 			(at 63.5 130.8099 0)
 			(effects
@@
 			)
 		)
-		(property "Value" "BDW93C"
+		(property "Value" "STN851-A"
 			(at 119.38 190.4999 0)
 			(effects
@@
 			)
 		)
-		(property "Value" "BDW93C"
+		(property "Value" "STN851-A"
 			(at 119.38 160.0199 0)
 			(effects
@@
 			)
 		)
-		(property "Value" "BDW93C"
+		(property "Value" "STN851-A"
 			(at 120.65 96.5199 0)
 			(effects
@@
 			)
 		)
-		(property "Value" "BDW93C"
+		(property "Value" "STN851-A"
 			(at 237.49 35.5599 0)
 			(effects
@@
 			)
 		)
-		(property "Value" "BDW93C"
+		(property "Value" "STN851-A"
 			(at 63.5 162.5599 0)
 			(effects
@@
 			)
 		)
-		(property "Value" "BDW93C"
+		(property "Value" "STN851-A"
 			(at 62.23 193.0399 0)
 			(effects
@@
 			)
 		)
-		(property "Value" "BDW93C"
+		(property "Value" "STN851-A"
 			(at 120.65 66.0399 0)
 			(effects
@@
 			)
 		)
-		(property "Value" "BDW93C"
+		(property "Value" "STN851-A"
 			(at 237.49 97.7899 0)
 			(effects
@@
 			)
 		)
-		(property "Value" "BDW93C"
+		(property "Value" "STN851-A"
 			(at 237.49 67.3099 0)
 			(effects
@@
 			)
 		)
-		(property "Value" "BDW93C"
+		(property "Value" "STN851-A"
 			(at 119.38 126.9999 0)
 			(effects
@@
 			)
 		)
-		(property "Value" "BDW93C"
+		(property "Value" "STN851-A"
 			(at 64.77 67.3099 0)
 			(effects

Commit message: began getting images for schematic appendix
Other:
- title: (none) -> A-Slave Solenoid Array
Changed lines of the file:
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@@
 	(generator_version "8.0")
 	(paper "A")
+	(title_block
+		(title "A-Slave Solenoid Array")
+		(date "2024-12-10")
+		(rev "A")
+	)
 	(junction
 		(at 60.96 85.09)
