File: Midi Bass Sch/DSolenoidA.kicad_sch (KiCad schematic)
At the start: 105 parts, among them Q53 STN851-A, Q54 STN851-A, Q55 STN851-A, Q56 STN851-A, Q57 STN851-A, Q58 STN851-A, Q59 STN851-A, Q60 STN851-A, Q61 STN851-A, Q62 STN851-A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

Commit message: began getting images for schematic appendix
Other:
- title: (none) -> D-Slave Solenoid Array
Changed lines of the file:
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@@
 	(generator_version "8.0")
 	(paper "A")
+	(title_block
+		(title "D-Slave Solenoid Array")
+		(date "2024-12-10")
+		(rev "A")
+	)
 	(junction
 		(at 237.49 24.13)
