File: Midi Bass Sch/GSolenoidA.kicad_sch (KiCad schematic)
At the start: 105 parts, among them Q73 STN851-A, Q74 STN851-A, Q75 STN851-A, Q76 STN851-A, Q77 STN851-A, Q78 STN851-A, Q79 STN851-A, Q80 STN851-A, Q81 STN851-A, Q82 STN851-A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

Commit message: began getting images for schematic appendix
Other:
- title: (none) -> G-Slave Solenoid Array
Changed lines of the file:
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@@
 	(generator_version "8.0")
 	(paper "A")
+	(title_block
+		(title "G-Slave Solenoid Array")
+		(date "2024-12-10")
+		(rev "A")
+	)
 	(junction
 		(at 69.85 21.59)
