File: Midi Bass Sch/Midi Bass Sch.kicad_pcb (KiCad board)
At the start: 2 copper layers, 251.5 x 142.2 mm, 550 parts, among them J2 Master ISCP, J3 E SLAVE ISCP, J4 A SLAVE ISCP, J5 A SLAVE ISCP, J6 D SLAVE ISCP, J7 G SLAVE ISCP, Q1 BDW93C, Q10 BDW93C, Q11 BDW93C, Q12 BDW93C, Q13 BDW93C, Q14 BDW93C, Q15 BDW93C, Q16 BDW93C, Q17 BDW93C, Q18 BDW93C, Q19 BDW93C, Q2 BDW93C, Q20 BDW93C, Q21 BDW93C, Q22 BDW93C, Q23 BDW93C, Q24 BDW93C, Q25 BDW93C, Q26 BDW93C, Q27 BDW93C, Q28 BDW93C, Q29 BDW93C, Q3 BDW93C, Q30 BDW93C, Q31 BDW93C, Q32 BDW93C, Q33 BDW93C, Q34 BDW93C, Q35 BDW93C, Q36 BDW93C, Q37 BDW93C, Q38 BDW93C, Q39 BDW93C, Q4 BDW93C, Q40 BDW93C, Q41 BDW93C, Q42 BDW93C, Q43 BDW93C, Q44 BDW93C, Q45 BDW93C, Q46 BDW93C, Q47 BDW93C, Q48 BDW93C, Q49 BDW93C, Q5 BDW93C, Q50 BDW93C, Q51 BDW93C, Q52 BDW93C, Q53 BDW93C, Q54 BDW93C, Q55 BDW93C, Q56 BDW93C, Q57 BDW93C, Q58 BDW93C, Q59 BDW93C, Q6 BDW93C, Q60 BDW93C, Q61 BDW93C, Q62 BDW93C, Q63 BDW93C, Q64 BDW93C, Q65 BDW93C, Q66 BDW93C, Q67 BDW93C, Q68 BDW93C, Q69 BDW93C, Q7 BDW93C, Q70 BDW93C, Q71 BDW93C, Q72 BDW93C, Q73 BDW93C, Q74 BDW93C, Q75 BDW93C, Q76 BDW93C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

Commit message: started basic pcb layout for Master pic
Parts:
- C2, D8, R15, R16, U2: moved to B.Cu
- moved L10 357.0 mm to (200.7, 153.1)
- moved L11 357.0 mm to (205.4, 153.1)
- moved L12 357.0 mm to (210.0, 153.1)
- moved L13 357.0 mm to (214.7, 153.1)
- moved L14 357.0 mm to (196.1, 160.3)
- moved L15 357.0 mm to (200.7, 160.3)
- moved L16 357.0 mm to (205.4, 160.3)
- moved L17 357.0 mm to (210.0, 160.3)
- moved L18 357.0 mm to (214.7, 160.3)
- moved L19 357.0 mm to (196.1, 167.5)
- moved L20 357.0 mm to (200.7, 167.5)
- moved L21 357.0 mm to (205.4, 167.5)
- moved L22 357.0 mm to (210.0, 167.5)
- moved L23 357.0 mm to (214.7, 167.5)
- moved L24 357.0 mm to (196.1, 174.7)
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Connections:
- D11 pad 1: Net-(C3-Pad1) -> MSCLR P
- D11 pad 2: MSCLR P -> Net-(C3-Pad1)
- D14 pad 1: Net-(C4-Pad1) -> MSCLR A
- D14 pad 2: MSCLR A -> Net-(C4-Pad1)
- D17 pad 1: Net-(C5-Pad1) -> MSCLR D
- D17 pad 2: MSCLR D -> Net-(C5-Pad1)
- D20 pad 1: Net-(C6-Pad1) -> MSCLR G
- D20 pad 2: MSCLR G -> Net-(C6-Pad1)
- D5 pad 1: Net-(C1-Pad1) -> Net-(U1-RE3/~{MCLR}/Vpp)
- D5 pad 2: Net-(U1-RE3/~{MCLR}/Vpp) -> Net-(C1-Pad1)
- D8 pad 1: Net-(C2-Pad1) -> MSCLR E
- D8 pad 2: MSCLR E -> Net-(C2-Pad1)

Commit message: began working on pcb layout deleted extra schematics for solenoid break out board
Parts:
- removed the L29 at (-94.4, 122.6)
- removed the L30 at (-89.8, 122.6)
- removed the L31 at (-85.1, 122.6)
- removed the L32 at (-80.5, 122.6)
- removed L34, L35, L36, L37, L38, L39, L40, L41, L42, L43, L44, L45, L46, L47, L48, L49, L50, L51, L52, L53, L54, L55, L56, L57, L58, L59, L60, L61, L62, L63, L64, L65, L66, L67, L68, L69, L70, L71, L72, L73, L74, L75, L76, L77, L78, L79, L80, L81, L82, L83, L84, L85, L86, L87, L88: Solenoid, Connector_PinHeader_2.54mm:PinHeader_1x02_P2.54mm_Vertical
- removed the Q29 at (-128.2, 91.8)
- removed the Q30 at (-128.2, 97.7)
- removed the Q31 at (-128.2, 103.7)
- removed the Q32 at (-128.2, 109.7)
- removed Q33, Q34, Q35, Q36, Q37, Q38, Q39, Q40, Q41, Q42, Q43, Q44, Q45, Q46, Q47, Q48, Q49, Q50, Q51, Q52, Q53, Q54, Q55, Q56, Q57, Q58, Q59, Q60, Q61, Q62, Q63, Q64, Q65, Q66, Q67, Q68, Q69, Q70, Q71, Q72, Q73, Q74, Q75, Q76, Q77, Q78, Q79, Q80, Q81, Q82, Q83, Q84, Q85, Q86, Q87, Q88: BDW93C, Package_TO_SOT_THT:TO-220-3_Vertical
- removed the R118 at (-94.4, 89.3)
- removed the R119 at (-94.4, 92.3)
- removed the R120 at (-94.4, 95.2)
- removed the R121 at (-94.4, 98.2)
- removed the R122 at (-94.4, 101.1)
- removed the R123 at (-94.4, 104.1)
- removed the R124 at (-94.4, 107.0)
- removed the R125 at (-94.4, 110.0)
- removed the R126 at (-94.4, 112.9)
- removed the R127 at (-94.4, 115.9)
- removed the R128 at (-94.4, 118.8)
- removed the R129 at (-89.6, 89.3)
- removed R130, R131, R132, R133, R134, R135, R142, R143, R144, R145, R146, R147, R148, R149, R150, R151, R152, R153, R158, R159, R160, R161, R162, R163, R164, R165, R170, R171, R172, R173, R174, R175, R176, R177, R184, R185, R186, R187, R188, R189, R190, R191, R192, R193, R194, R195, R202, R203, R204, R205, R206, R207, R208, R209, R210, R211, R212, R213, R218, R219, R220, R221, R222, R223, R224, R225, R230, R231, R232, R233, R234, R235, R236, R237, R244, R245, R246, R247, R248, R249, R250, R251, R252, R253, R254, R255, R262, R263, R264, R265, R266, R267, R268, R269, R270, R271, R272, R273, R278, R279, R280, R281, R282, R283, R284, R285, R290, R291, R292, R293, R294, R295, R296, R297: 1kΩ, Resistor_SMD:R_0805_2012Metric_Pad1.20x1.40mm_HandSolder
- removed R136, R137, R138, R139, R140, R141, R154, R155, R156, R157, R166, R167, R168, R169, R178, R179, R180, R181, R182, R183, R196, R197, R198, R199, R200, R201, R214, R215, R216, R217, R226, R227, R228, R229, R238, R239, R240, R241, R242, R243, R256, R257, R258, R259, R260, R261, R274, R275, R276, R277, R286, R287, R288, R289: 4.7kΩ, Resistor_SMD:R_0805_2012Metric_Pad1.20x1.40mm_HandSolder
- removed the U14 at (-126.6, 81.9)
- removed the U15 at (-117.1, 81.9)
- removed U17, U18, U19, U20, U21, U22, U23, U24, U25, U26, U27, U28: LTV-247, Package_SO:SOP-16_4.4x10.4mm_P1.27mm
- added C10: 0.1uF, Capacitor_SMD:C_0805_2012Metric_Pad1.18x1.45mm_HandSolder, F.Cu at (31.2, 60.9)
- added C7: 100uF, Capacitor_THT:CP_Radial_D12.5mm_P2.50mm, F.Cu at (10.6, 52.4)
- added C8: 0.1uF, Capacitor_SMD:C_0805_2012Metric_Pad1.18x1.45mm_HandSolder, F.Cu at (31.2, 57.9)
- added C9: 100uF, Capacitor_THT:CP_Radial_D12.5mm_P2.50mm, F.Cu at (10.6, 66.5)
- added J11: A Slave OUT, Connector_PinHeader_2.54mm:PinHeader_1x21_P2.54mm_Vertical, F.Cu at (192.4, 110.5)
- added J13: D Slave OUT, Connector_PinHeader_2.54mm:PinHeader_1x21_P2.54mm_Vertical, F.Cu at (-85.7, -33.6)
- added J15: G Slave OUT, Connector_PinHeader_2.54mm:PinHeader_1x21_P2.54mm_Vertical, F.Cu at (150.5, 221.0)
- added J16: Power In, OF footprints:Two_Pin_Screw_Terminal, F.Cu at (25.9, 50.4)
- added J4: E Slave Out, Connector_PinHeader_2.54mm:PinHeader_1x21_P2.54mm_Vertical, F.Cu at (148.6, 110.5)
- added J5: Solenoid In, Connector_PinHeader_2.54mm:PinHeader_1x21_P2.54mm_Vertical, F.Cu at (149.9, 66.0)
- added J7: Pick Unit, Connector_PinHeader_2.54mm:PinHeader_1x10_P2.54mm_Vertical, F.Cu at (48.8, 10.6)
- added J8: Pluck Out, Connector_PinHeader_2.54mm:PinHeader_1x13_P2.54mm_Vertical, F.Cu at (44.1, 10.6)
- added J9: Pluck IN, Connector_PinHeader_2.54mm:PinHeader_1x13_P2.54mm_Vertical, F.Cu at (6.83, 10.6)
- added L10: Solenoid, Connector_PinHeader_2.54mm:PinHeader_1x02_P2.54mm_Vertical, F.Cu at (27.7, 22.6)
- added L11: Solenoid, Connector_PinHeader_2.54mm:PinHeader_1x02_P2.54mm_Vertical, F.Cu at (32.3, 22.6)
- added L12: Solenoid, Connector_PinHeader_2.54mm:PinHeader_1x02_P2.54mm_Vertical, F.Cu at (37.0, 22.6)
- added L9: Solenoid, Connector_PinHeader_2.54mm:PinHeader_1x02_P2.54mm_Vertical, F.Cu at (23.0, 22.6)
- added Q10: STN851-A, Package_TO_SOT_THT:TO-220-3_Vertical, F.Cu at (12.4, 18.2)
- added Q11: STN851-A, Package_TO_SOT_THT:TO-220-3_Vertical, F.Cu at (12.4, 24.2)
- added Q12: STN851-A, Package_TO_SOT_THT:TO-220-3_Vertical, F.Cu at (12.4, 30.1)
- added Q9: STN851-A, Package_TO_SOT_THT:TO-220-3_Vertical, F.Cu at (12.4, 12.2)
- added R46: 4.7kΩ, Resistor_SMD:R_0805_2012Metric_Pad1.20x1.40mm_HandSolder, F.Cu at (23.1, 28.9)
- added R47: 4.7kΩ, Resistor_SMD:R_0805_2012Metric_Pad1.20x1.40mm_HandSolder, F.Cu at (23.1, 31.9)
- added R48: 4.7kΩ, Resistor_SMD:R_0805_2012Metric_Pad1.20x1.40mm_HandSolder, F.Cu at (23.1, 34.8)
- added R49: 4.7kΩ, Resistor_SMD:R_0805_2012Metric_Pad1.20x1.40mm_HandSolder, F.Cu at (23.1, 37.8)
- added R50: 1kΩ, Resistor_SMD:R_0805_2012Metric_Pad1.20x1.40mm_HandSolder, F.Cu at (27.8, 28.9)
- added R51: 1kΩ, Resistor_SMD:R_0805_2012Metric_Pad1.20x1.40mm_HandSolder, F.Cu at (27.8, 31.9)
- added R52: 1kΩ, Resistor_SMD:R_0805_2012Metric_Pad1.20x1.40mm_HandSolder, F.Cu at (27.8, 34.8)
- added R53: 1kΩ, Resistor_SMD:R_0805_2012Metric_Pad1.20x1.40mm_HandSolder, F.Cu at (27.8, 37.8)
- added R54: 1kΩ, Resistor_SMD:R_0805_2012Metric_Pad1.20x1.40mm_HandSolder, F.Cu at (32.6, 28.9)
- added R55: 1kΩ, Resistor_SMD:R_0805_2012Metric_Pad1.20x1.40mm_HandSolder, F.Cu at (32.6, 31.9)
- added R56: 1kΩ, Resistor_SMD:R_0805_2012Metric_Pad1.20x1.40mm_HandSolder, F.Cu at (32.6, 34.8)
- added R57: 1kΩ, Resistor_SMD:R_0805_2012Metric_Pad1.20x1.40mm_HandSolder, F.Cu at (32.6, 37.8)
- added TP10: P-IN, Connector_PinHeader_2.54mm:PinHeader_1x01_P2.54mm_Vertical, F.Cu at (33.9, 47.7)
- added TP11: 5v, Connector_PinHeader_2.54mm:PinHeader_1x01_P2.54mm_Vertical, F.Cu at (33.9, 52.4)
- added U6: LTV-247, Package_SO:SOP-16_4.4x10.4mm_P1.27mm, F.Cu at (25.5, 14.3)
- added U7: LTV-247, Package_SO:SOP-16_4.4x10.4mm_P1.27mm, F.Cu at (35.0, 14.3)
- J6: renamed from J4; value A SLAVE ISCP -> Pluck ISCP
- L33: value Solenoid -> 10uH; footprint Connector_PinHeader_2.54mm:PinHeader_1x02_P2.54mm_Vertical -> Inductor_THT:L_Axial_L5.0mm_D3.6mm_P10.00mm_Horizontal_Murata_BL01RN1A2A2
- Q1, Q2, Q3, Q4, Q5, Q6, Q7, Q8: value BDW93C -> STN851-A
- Q13: renamed from Q9; value BDW93C -> STN851-A
- Q14: renamed from Q10; value BDW93C -> STN851-A
- Q15: renamed from Q11; value BDW93C -> STN851-A
- Q16: renamed from Q12; value BDW93C -> STN851-A
- Q17: renamed from Q13; value BDW93C -> STN851-A
- Q18: renamed from Q14; value BDW93C -> STN851-A
- Q19: renamed from Q15; value BDW93C -> STN851-A
- Q20: renamed from Q16; value BDW93C -> STN851-A
- Q21: renamed from Q17; value BDW93C -> STN851-A
- Q22: renamed from Q18; value BDW93C -> STN851-A
- Q23: renamed from Q19; value BDW93C -> STN851-A
- Q24: renamed from Q20; value BDW93C -> STN851-A
- Q25: renamed from Q21; value BDW93C -> STN851-A
- Q26: renamed from Q22; value BDW93C -> STN851-A
- Q27: renamed from Q23; value BDW93C -> STN851-A
- Q28: renamed from Q24; value BDW93C -> STN851-A
- Q29: renamed from Q25; value BDW93C -> STN851-A
- Q30: renamed from Q26; value BDW93C -> STN851-A
- Q31: renamed from Q27; value BDW93C -> STN851-A
- Q32: renamed from Q28; value BDW93C -> STN851-A
- U10: renamed from U8; footprint Package_DFN_QFN:TQFN-44-1EP_7x7mm_P0.5mm_EP4.7x4.7mm -> OF footprints:TQFN-44_7x7_Pitch0.4mm; moved to B.Cu
- U16: value LTV-247 -> LM1117MP-1.8; footprint Package_SO:SOP-16_4.4x10.4mm_P1.27mm -> Package_TO_SOT_SMD:SOT-223-3_TabPin2
- U2, U3: footprint Package_DFN_QFN:TQFN-44-1EP_7x7mm_P0.5mm_EP4.7x4.7mm -> OF footprints:TQFN-44_7x7_Pitch0.4mm
- U8: renamed from U6; footprint Package_DFN_QFN:TQFN-44-1EP_7x7mm_P0.5mm_EP4.7x4.7mm -> OF footprints:TQFN-44_7x7_Pitch0.4mm
- U9: renamed from U7; footprint Package_DFN_QFN:TQFN-44-1EP_7x7mm_P0.5mm_EP4.7x4.7mm -> OF footprints:TQFN-44_7x7_Pitch0.4mm
- moved R59 297.8 mm to (227.0, 135.3)
- moved C4 286.6 mm to (222.5, 132.7), turned to 180 degrees
- moved R58 285.1 mm to (216.2, 123.8)
- moved SW4 284.1 mm to (219.6, 124.4)
- moved TP7 282.6 mm to (214.6, 116.2)
- moved R60 282.6 mm to (211.8, 135.9), turned to 180 degrees
- moved D14 282.1 mm to (222.5, 135.3)
- moved R61 277.0 mm to (206.6, 136.5)
- moved U8 273.1 mm to (208.9, 127.6)
- moved D15 271.9 mm to (211.7, 139.1)
- moved D16 266.1 mm to (206.6, 139.1), turned to 180 degrees
- moved J10 264.7 mm to (191.1, 121.9)
- moved R69 260.7 mm to (135.3, 208.6), turned to 90 degrees
- moved R68 259.0 mm to (130.2, 208.6), turned to 90 degrees
- moved D22 250.7 mm to (135.3, 213.1), turned to 90 degrees
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- renumbered D2 to D1, D1 to D2, J5 to J10, J6 to J12, J7 to J14, L9 to L13, L10 to L14, L11 to L15, L12 to L16, L13 to L17, L14 to L18, L15 to L19, L16 to L20, L17 to L21, L18 to L22, L19 to L23, L20 to L24, L21 to L25, L22 to L26, L23 to L27, L24 to L28, L25 to L29, L26 to L30, L27 to L31, L28 to L32, R88 to R100, R89 to R101, R90 to R102, R91 to R103, R92 to R104, R93 to R105, R94 to R106, R95 to R107, R96 to R108, R97 to R109, R98 to R110, R99 to R111, R100 to R112, R101 to R113, R102 to R114, R103 to R115, R104 to R116, R105 to R117, R106 to R118, R107 to R119, R108 to R120, R109 to R121, R110 to R122, R111 to R123, R112 to R124, R113 to R125, R114 to R126, R115 to R127, R116 to R128, R117 to R129, R3 to R2, R2 to R3, R46 to R58, R47 to R59, R48 to R60, R49 to R61, R50 to R62, R51 to R63, R52 to R64, R53 to R65, R54 to R66, R55 to R67, R56 to R68, R57 to R69, R58 to R70, R59 to R71, R60 to R72, R61 to R73, R62 to R74, R63 to R75, R64 to R76, R65 to R77, R66 to R78, R67 to R79, R68 to R80, R69 to R81, R70 to R82, R71 to R83, R72 to R84, R73 to R85, R74 to R86, R75 to R87, R76 to R88, R77 to R89, R78 to R90, R79 to R91, R80 to R92, R81 to R93, R82 to R94, R83 to R95, R84 to R96, R85 to R97, R86 to R98, R87 to R99, U9 to U11, U10 to U12, U11 to U13, U12 to U14, U13 to U15
Connections:
- J10 pad 4: F2 -> RB7 A
- J10 pad 5: E2 -> RB6 A
- J12 pad 4: A#2 -> RB7 D
- J12 pad 5: A2 -> RB6 D
- J14 pad 4: D#3 -> RB7 G
- J14 pad 5: D3 -> RB6 G
- J6 pad 4: G1 -> RB7 P
- J6 pad 5: G0 -> RB6 P
- L33 pad 1: +12v -> Net-(U16-VO)
- L33 pad 2: Net-(Q33-C) -> +5v
- R20 pad 2: Net-(U3-RC1/T1OSI/CCP2) -> Net-(U3-RD7/C4OUT/PSMC3C)
- R21 pad 1: Net-(D13-A) -> Net-(U3-RD6/PSMC3D)
- R21 pad 2: Net-(U3-RC0/T1CKI/PSMC1A) -> Net-(D13-A)
- U10 pad 1: A3 -> unconnected-(U10-RC7/RX/DT/C4Out-Pad1)
- U10 pad 10: A#2 -> Net-(U10-RB2/AN8/OPA2IN-/DAC3OUT1)
- U10 pad 11: B2 -> Net-(U10-RB3/AN9/CXNI2-/CCP2)
- U10 pad 14: C3 -> Net-(U10-RB4/AN11/C3IN1+)
- U10 pad 15: C#3 -> Net-(U10-RB5/AN13/C4IN2-/CCP3)
- U10 pad 16: D3 -> RB6 A
- U10 pad 17: D#3 -> RB7 A
- U10 pad 19: unconnected-(U8-RA0/AN0/CxIN0--Pad19) -> Net-(U10-RA0/AN0/CxIN0-)
- U10 pad 2: D4 -> Net-(U10-RD4/PSM3F)
- U10 pad 20: unconnected-(U8-RA1/AN1/CxIN1-/OPA1OUT-Pad20) -> Net-(U10-RA1/AN1/CxIN1-/OPA1OUT)
- U10 pad 21: unconnected-(U8-RA2/AN2/CxIN0+/DAC1OUT1-Pad21) -> Net-(U10-RA2/AN2/CxIN0+/DAC1OUT1)
- U10 pad 22: unconnected-(U8-RA3/AN3/VREF+/C1IN1+-Pad22) -> Net-(U10-RA3/AN3/VREF+/C1IN1+)
- U10 pad 23: unconnected-(U8-RA4/C1OUT/OPA1IN+/T0CKI-Pad23) -> Net-(U10-RA4/C1OUT/OPA1IN+/T0CKI)
- U10 pad 24: unconnected-(U8-RA5/AN4/C2OUT/OPA1IN+-Pad24) -> Net-(U10-RA5/AN4/C2OUT/OPA1IN+)
- U10 pad 3: D#4 -> Net-(U10-RD5/PSMC3E)
- U10 pad 32: E3 -> unconnected-(U10-RC0/T1CKI/PSMC1A-Pad32)
- U10 pad 35: F3 -> unconnected-(U10-RC1/T1OSI/CCP2-Pad35)
- U10 pad 36: F#3 -> unconnected-(U10-RC2/CCP1/PSMC1C-Pad36)
- U10 pad 38: A#3 -> Net-(U10-RD0/OPA3IN+)
- U10 pad 39: B3 -> Net-(U10-RD1/CxIN4-/OPA3OUT)
- U10 pad 40: C4 -> Net-(U10-RD2/OPA3IN-/DAC4OUT1)
- U10 pad 41: C#4 -> Net-(U10-RD3/PSMC4A)
- U10 pad 43: G3 -> unconnected-(U10-RC5/SDO/PSMC1F-Pad43)
- U10 pad 44: G#3 -> unconnected-(U10-RC6/TX/CK/PSMC2A-Pad44)
- U10 pad 8: G#2 -> Net-(U10-RB0/AN12/CCP1/C2IN1+)
- U10 pad 9: A2 -> Net-(U10-RB1/AN10/CxIN3-/OPA2OUT)
- U16 pad 1: F#2 -> Earth_GND
- U16 pad 2: Net-(R141-Pad2) -> Net-(U16-VO)
- U16 pad 3: G2 -> +12v
- U2 pad 1: F#2 -> unconnected-(U2-RC7/RX/DT/C4Out-Pad1)
- U2 pad 19: unconnected-(U2-RA0/AN0/CxIN0--Pad19) -> C#2
- U2 pad 20: unconnected-(U2-RA1/AN1/CxIN1-/OPA1OUT-Pad20) -> D2
- U2 pad 21: unconnected-(U2-RA2/AN2/CxIN0+/DAC1OUT1-Pad21) -> D#2
- U2 pad 22: unconnected-(U2-RA3/AN3/VREF+/C1IN1+-Pad22) -> E2
- U2 pad 23: unconnected-(U2-RA4/C1OUT/OPA1IN+/T0CKI-Pad23) -> F2
- U2 pad 24: unconnected-(U2-RA5/AN4/C2OUT/OPA1IN+-Pad24) -> F#2
- U2 pad 32: C#2 -> unconnected-(U2-RC0/T1CKI/PSMC1A-Pad32)
- U2 pad 35: D2 -> unconnected-(U2-RC1/T1OSI/CCP2-Pad35)
- U2 pad 36: D#2 -> unconnected-(U2-RC2/CCP1/PSMC1C-Pad36)
- U2 pad 43: E2 -> unconnected-(U2-RC5/SDO/PSMC1F-Pad43)
- U2 pad 44: F2 -> unconnected-(U2-RC6/TX/CK/PSMC2A-Pad44)
- U3 pad 10: A0 -> /String Strike Slave/A0
- U3 pad 11: A1 -> /String Strike Slave/A1
- U3 pad 14: D0 -> /String Strike Slave/D0
- U3 pad 15: D1 -> /String Strike Slave/D1
- U3 pad 16: G0 -> RB6 P
- U3 pad 17: G1 -> RB7 P
- U3 pad 19: unconnected-(U3-RA0/AN0/CxIN0--Pad19) -> Net-(U3-RA0/AN0/CxIN0-)
- U3 pad 20: unconnected-(U3-RA1/AN1/CxIN1-/OPA1OUT-Pad20) -> Net-(U3-RA1/AN1/CxIN1-/OPA1OUT)
- U3 pad 21: unconnected-(U3-RA2/AN2/CxIN0+/DAC1OUT1-Pad21) -> Net-(U3-RA2/AN2/CxIN0+/DAC1OUT1)
- U3 pad 22: unconnected-(U3-RA3/AN3/VREF+/C1IN1+-Pad22) -> Net-(U3-RA3/AN3/VREF+/C1IN1+)
- U3 pad 23: unconnected-(U3-RA4/C1OUT/OPA1IN+/T0CKI-Pad23) -> Net-(U3-RA4/C1OUT/OPA1IN+/T0CKI)
- U3 pad 24: unconnected-(U3-RA5/AN4/C2OUT/OPA1IN+-Pad24) -> Net-(U3-RA5/AN4/C2OUT/OPA1IN+)
- U3 pad 26: unconnected-(U3-RE1/AN6/PSMC3B-Pad26) -> Net-(U3-RE1/AN6/PSMC3B)
- U3 pad 27: unconnected-(U3-RE2/AN7/PSMC3A-Pad27) -> Net-(U3-RE2/AN7/PSMC3A)
- U3 pad 32: Net-(U3-RC0/T1CKI/PSMC1A) -> unconnected-(U3-RC0/T1CKI/PSMC1A-Pad32)
- U3 pad 35: Net-(U3-RC1/T1OSI/CCP2) -> unconnected-(U3-RC1/T1OSI/CCP2-Pad35)
- U3 pad 38: unconnected-(U3-RD0/OPA3IN+-Pad38) -> /String Strike Slave/E MUTE
- U3 pad 39: unconnected-(U3-RD1/CxIN4-/OPA3OUT-Pad39) -> /String Strike Slave/A MUTE
- U3 pad 4: unconnected-(U3-RD6/PSMC3D-Pad4) -> Net-(U3-RD6/PSMC3D)
- U3 pad 40: unconnected-(U3-RD2/OPA3IN-/DAC4OUT1-Pad40) -> /String Strike Slave/D MUTE
- U3 pad 41: unconnected-(U3-RD3/PSMC4A-Pad41) -> /String Strike Slave/G MUTE
- U3 pad 5: unconnected-(U3-RD7/C4OUT/PSMC3C-Pad5) -> Net-(U3-RD7/C4OUT/PSMC3C)
- U3 pad 8: E0 -> /String Strike Slave/E0
- U3 pad 9: E1 -> /String Strike Slave/E1
- U8 pad 1: B2 -> unconnected-(U8-RC7/RX/DT/C4Out-Pad1)
- U8 pad 10: C2 -> Net-(U8-RB2/AN8/OPA2IN-/DAC3OUT1)
- U8 pad 11: C#2 -> Net-(U8-RB3/AN9/CXNI2-/CCP2)
- U8 pad 14: D2 -> Net-(U8-RB4/AN11/C3IN1+)
- U8 pad 15: D#2 -> Net-(U8-RB5/AN13/C4IN2-/CCP3)
- U8 pad 16: E2 -> RB6 A
- U8 pad 17: F2 -> RB7 A
- U8 pad 19: unconnected-(U6-RA0/AN0/CxIN0--Pad19) -> Net-(U8-RA0/AN0/CxIN0-)
- U8 pad 2: E3 -> Net-(U8-RD4/PSM3F)
- U8 pad 20: unconnected-(U6-RA1/AN1/CxIN1-/OPA1OUT-Pad20) -> Net-(U8-RA1/AN1/CxIN1-/OPA1OUT)
- U8 pad 21: unconnected-(U6-RA2/AN2/CxIN0+/DAC1OUT1-Pad21) -> Net-(U8-RA2/AN2/CxIN0+/DAC1OUT1)
- U8 pad 22: unconnected-(U6-RA3/AN3/VREF+/C1IN1+-Pad22) -> Net-(U8-RA3/AN3/VREF+/C1IN1+)
- U8 pad 23: unconnected-(U6-RA4/C1OUT/OPA1IN+/T0CKI-Pad23) -> Net-(U8-RA4/C1OUT/OPA1IN+/T0CKI)
- U8 pad 24: unconnected-(U6-RA5/AN4/C2OUT/OPA1IN+-Pad24) -> Net-(U8-RA5/AN4/C2OUT/OPA1IN+)
- U8 pad 3: F3 -> Net-(U8-RD5/PSMC3E)
- U8 pad 32: F#2 -> unconnected-(U8-RC0/T1CKI/PSMC1A-Pad32)
- U8 pad 35: G2 -> unconnected-(U8-RC1/T1OSI/CCP2-Pad35)
- U8 pad 36: G#2 -> unconnected-(U8-RC2/CCP1/PSMC1C-Pad36)
- U8 pad 38: C3 -> Net-(U8-RD0/OPA3IN+)
- U8 pad 39: C#3 -> Net-(U8-RD1/CxIN4-/OPA3OUT)
- U8 pad 40: D3 -> Net-(U8-RD2/OPA3IN-/DAC4OUT1)
- U8 pad 41: D#3 -> Net-(U8-RD3/PSMC4A)
- U8 pad 43: A2 -> unconnected-(U8-RC5/SDO/PSMC1F-Pad43)
- U8 pad 44: A#2 -> unconnected-(U8-RC6/TX/CK/PSMC2A-Pad44)
- U8 pad 8: A#1 -> Net-(U8-RB0/AN12/CCP1/C2IN1+)
- U8 pad 9: B1 -> Net-(U8-RB1/AN10/CxIN3-/OPA2OUT)
- U9 pad 1: E3 -> unconnected-(U9-RC7/RX/DT/C4Out-Pad1)
- U9 pad 10: F2 -> Net-(U9-RB2/AN8/OPA2IN-/DAC3OUT1)
- U9 pad 11: F#2 -> Net-(U9-RB3/AN9/CXNI2-/CCP2)
- U9 pad 14: G2 -> Net-(U9-RB4/AN11/C3IN1+)
- U9 pad 15: G#2 -> Net-(U9-RB5/AN13/C4IN2-/CCP3)
- U9 pad 16: A2 -> RB6 D
- U9 pad 17: A#2 -> RB7 D
- U9 pad 19: unconnected-(U7-RA0/AN0/CxIN0--Pad19) -> Net-(U9-RA0/AN0/CxIN0-)
- U9 pad 2: A3 -> Net-(U9-RD4/PSM3F)
- U9 pad 20: unconnected-(U7-RA1/AN1/CxIN1-/OPA1OUT-Pad20) -> Net-(U9-RA1/AN1/CxIN1-/OPA1OUT)
- U9 pad 21: unconnected-(U7-RA2/AN2/CxIN0+/DAC1OUT1-Pad21) -> Net-(U9-RA2/AN2/CxIN0+/DAC1OUT1)
- U9 pad 22: unconnected-(U7-RA3/AN3/VREF+/C1IN1+-Pad22) -> Net-(U9-RA3/AN3/VREF+/C1IN1+)
- U9 pad 23: unconnected-(U7-RA4/C1OUT/OPA1IN+/T0CKI-Pad23) -> Net-(U9-RA4/C1OUT/OPA1IN+/T0CKI)
- U9 pad 24: unconnected-(U7-RA5/AN4/C2OUT/OPA1IN+-Pad24) -> Net-(U9-RA5/AN4/C2OUT/OPA1IN+)
- U9 pad 3: A#3 -> Net-(U9-RD5/PSMC3E)
- U9 pad 32: B2 -> unconnected-(U9-RC0/T1CKI/PSMC1A-Pad32)
- U9 pad 35: C3 -> unconnected-(U9-RC1/T1OSI/CCP2-Pad35)
- U9 pad 36: C#3 -> unconnected-(U9-RC2/CCP1/PSMC1C-Pad36)
- U9 pad 38: F3 -> Net-(U9-RD0/OPA3IN+)
- U9 pad 39: F#3 -> Net-(U9-RD1/CxIN4-/OPA3OUT)
- U9 pad 40: G3 -> Net-(U9-RD2/OPA3IN-/DAC4OUT1)
- U9 pad 41: G#3 -> Net-(U9-RD3/PSMC4A)
- U9 pad 43: D3 -> unconnected-(U9-RC5/SDO/PSMC1F-Pad43)
- U9 pad 44: D#3 -> unconnected-(U9-RC6/TX/CK/PSMC2A-Pad44)
- U9 pad 8: D#2 -> Net-(U9-RB0/AN12/CCP1/C2IN1+)
- U9 pad 9: E2 -> Net-(U9-RB1/AN10/CxIN3-/OPA2OUT)
Routing:
- net GND: track 0.00 -> 157.7 mm
- net +5v: track 0.00 -> 115.2 mm, vias 0 -> 1
- net RB7 A: track 0.00 -> 65.7 mm, vias 0 -> 1
- net Net-(U8-RD5/PSMC3E): track 0.00 -> 64.3 mm
- net G#1: track 0.00 -> 60.4 mm
- net Net-(U8-RD4/PSM3F): track 0.00 -> 60.3 mm
- net RB6 A: track 0.00 -> 58.9 mm, vias 0 -> 1
- net G1: track 0.00 -> 53.7 mm
- net F#1: track 0.00 -> 45.4 mm
- net Net-(U1-RE3/~{MCLR}/Vpp): track 0.00 -> 44.5 mm, vias 0 -> 1
- net RB6M: track 0.00 -> 43.7 mm, vias 0 -> 1
- net Net-(U8-RD3/PSMC4A): track 0.00 -> 40.5 mm
- net Net-(U1-RC0/T1OSO/T1CK1): track 0.00 -> 39.0 mm
- net F1: track 0.00 -> 38.1 mm
- net Net-(U10-RB0/AN12/CCP1/C2IN1+): track 0.00 -> 37.4 mm
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
Commit message: added traces for D processor began Pluck processor
Parts:
- U3, U9: moved to B.Cu
- moved J13 424.5 mm to (254.0, 221.0), turned to -90 degrees
- moved R65 357.9 mm to (240.0, 207.4), turned to 90 degrees
- moved R64 355.3 mm to (234.9, 207.3), turned to 90 degrees
- moved D19 347.2 mm to (240.0, 211.2), turned to 90 degrees
- moved TP8 345.9 mm to (222.2, 214.6)
- moved D18 344.6 mm to (234.9, 211.1), turned to 90 degrees
- moved U9 343.1 mm to (228.0, 208.3), turned to -90 degrees
- moved C5 341.1 mm to (231.4, 196.8)
- moved D17 336.9 mm to (231.4, 199.4), turned to 180 degrees
- moved R63 334.6 mm to (215.0, 196.8), turned to 180 degrees
- moved SW5 334.1 mm to (220.2, 192.3)
- moved R62 333.4 mm to (215.0, 191.8)
- moved J12 332.3 mm to (203.2, 200.7)
- moved J7 292.1 mm to (287.0, 179.7)
- moved J6 286.8 mm to (254.9, 153.4)
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Routing:
- net GND: track 157.7 -> 281.6 mm
- net RB6 D: track 0.00 -> 59.1 mm
- net +5v: track 115.2 -> 173.8 mm
- net RB7 P: track 0.00 -> 56.5 mm
- net RB7 D: track 0.00 -> 54.7 mm
- net RB6 P: track 0.00 -> 50.7 mm
- net /String Strike Slave/E0: track 0.00 -> 48.1 mm
- net /String Strike Slave/E1: track 0.00 -> 46.8 mm
- net /String Strike Slave/A0: track 0.00 -> 45.6 mm
- net /String Strike Slave/A1: track 0.00 -> 44.3 mm
- net /String Strike Slave/D0: track 0.00 -> 43.9 mm
- net /String Strike Slave/D1: track 0.00 -> 43.8 mm
- net MSCLR D: track 0.00 -> 36.3 mm
- net Net-(U9-RB0/AN12/CCP1/C2IN1+): track 0.00 -> 35.8 mm
- net Net-(U9-RD5/PSMC3E): track 0.00 -> 35.1 mm
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
Commit message: created pcb for breakout working on pcb for main control board
Parts:
- removed J5: Solenoid In, Connector_PinHeader_2.54mm:PinHeader_1x21_P2.54mm_Vertical
- removed J9: Pluck IN, Connector_PinHeader_2.54mm:PinHeader_1x13_P2.54mm_Vertical
- removed L1, L10, L11, L12, L13, L14, L15, L16, L17, L18, L19, L2, L20, L21, L22, L23, L24, L25, L26, L27, L28, L29, L3, L30, L31, L32, L4, L5, L6, L7, L8, L9: Solenoid, Connector_PinHeader_2.54mm:PinHeader_1x02_P2.54mm_Vertical
- removed Q1, Q10, Q11, Q12, Q13, Q14, Q15, Q16, Q17, Q18, Q19, Q2, Q20, Q21, Q22, Q23, Q24, Q25, Q26, Q27, Q28, Q29, Q3, Q30, Q31, Q32, Q4, Q5, Q6, Q7, Q8, Q9: STN851-A, Package_TO_SOT_THT:TO-220-3_Vertical
- removed R100, R101, R102, R103, R104, R105, R110, R111, R112, R113, R114, R115, R116, R117, R122, R123, R124, R125, R126, R127, R128, R129, R26, R27, R28, R29, R30, R31, R32, R33, R38, R39, R40, R41, R42, R43, R44, R45, R50, R51, R52, R53, R54, R55, R56, R57, R76, R77, R78, R79, R80, R81, R82, R83, R84, R85, R86, R87, R94, R95, R96, R97, R98, R99: 1kΩ, Resistor_SMD:R_0805_2012Metric_Pad1.20x1.40mm_HandSolder
- removed R106, R107, R108, R109, R118, R119, R120, R121, R22, R23, R24, R25, R34, R35, R36, R37, R46, R47, R48, R49, R70, R71, R72, R73, R74, R75, R88, R89, R90, R91, R92, R93: 4.7kΩ, Resistor_SMD:R_0805_2012Metric_Pad1.20x1.40mm_HandSolder
- removed U11, U12, U13, U14, U15, U4, U5, U6, U7: LTV-247, Package_SO:SOP-16_4.4x10.4mm_P1.27mm
- added POWER OUT: Two_Pin_Screw_Terminal, OF Footprints:Two_Pin_Screw_Terminal, F.Cu at (247.0, 194.9)
- C10, C8: moved to B.Cu
- moved C7 262.8 mm to (225.5, 203.8)
- moved J16 262.3 mm to (227.3, 218.4)
- moved C9 247.1 mm to (225.5, 188.6)
- moved C8 246.5 mm to (226.9, 207.6)
- moved U16 244.6 mm to (215.9, 212.1), turned to 90 degrees
- moved TP10 240.6 mm to (215.9, 205.1)
- moved L33 237.3 mm to (215.9, 201.8), turned to 90 degrees
- moved C10 231.7 mm to (226.9, 184.8)
- moved TP11 227.0 mm to (215.9, 188.0)
- moved J7 45.5 mm to (247.7, 156.8)
- moved C5 41.9 mm to (189.5, 196.8)
- moved D17 41.9 mm to (189.5, 199.3)
- moved D18 41.9 mm to (193.0, 211.0)
- moved D19 41.9 mm to (198.1, 211.1)
- moved J12 41.9 mm to (161.3, 200.6)
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Routing:
- net +12v: track 0.00 -> 63.3 mm
- net Earth_GND: track 0.00 -> 61.6 mm
- net GND: track 281.6 -> 308.7 mm
- net MSCLR A: track 16.4 -> 43.5 mm, vias 0 -> 1
- net +5v: track 173.8 -> 191.5 mm
- net Net-(U16-VO): track 0.00 -> 9.92 mm
Other:
- board size 251.5 x 142.2 mm -> 161.9 x 116.8 mm
- board text added: "+"

Commit message: working in finishing Rev A pcb for motherboard
Parts:
- removed POWER OUT: Two_Pin_Screw_Terminal, OF Footprints:Two_Pin_Screw_Terminal
- added ?: , , F.Cu at (253.4, 112.4)
- added ?: , , F.Cu at (89.5, 112.4)
- added ?: , , F.Cu at (253.4, 219.1)
- added G***: LOGO, Logos:Wisteria Logo .75x.75, F.Cu at (100.5, 151.8)
- added G***: LOGO, Logos:ISU 1inch, F.Cu at (102.5, 165.3)
- added G***: LOGO, Logos:Bengal Head .5x.5, F.Cu at (118.0, 153.7)
- added Power Out: Two_Pin_Screw_Terminal, OF Footprints:Two_Pin_Screw_Terminal, F.Cu at (252.7, 194.9)
- added R110: 10Ω, Resistor_SMD:R_0805_2012Metric_Pad1.20x1.40mm_HandSolder, F.Cu at (226.1, 135.0)
- added REF**: 6-32 Mount, OF Footprints:6-32 Mount, F.Cu at (89.5, 219.1)
- added SW7: Pluck Reset, Button_Switch_THT:SW_PUSH_6mm_H5mm, F.Cu at (214.6, 131.7)
- C2, D8, R15, R16, U2: moved to F.Cu
- moved J2 63.1 mm to (179.1, 167.3), turned to 0 degrees
- moved D7 62.9 mm to (178.4, 159.6), turned to 180 degrees
- moved TP1 61.0 mm to (171.4, 174.9), turned to 90 degrees
- moved TP2 58.3 mm to (157.5, 182.5), turned to 90 degrees
- moved R12 57.9 mm to (163.5, 178.7), turned to 0 degrees
- moved R14 57.6 mm to (174.6, 159.6), turned to 180 degrees
- moved C1 56.9 mm to (151.6, 183.5), turned to -90 degrees
- moved R5 55.8 mm to (148.6, 183.5), turned to -90 degrees
- moved R2 54.4 mm to (168.6, 171.1), turned to 0 degrees
- moved TP3 53.7 mm to (163.8, 174.9), turned to 90 degrees
- moved J11 51.8 mm to (212.1, 110.5), turned to -90 degrees
- moved D5 51.7 mm to (151.6, 179.7), turned to -90 degrees
- moved R1 50.5 mm to (148.6, 179.7), turned to -90 degrees
- moved D1 49.8 mm to (164.1, 171.1), turned to 0 degrees
- moved J10 49.6 mm to (208.3, 127.0)
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Connections:
- J15 pad 7: RB6 A -> RB6 G
- J15 pad 8: RB7 A -> RB7 G
- U10 pad 16: RB6 A -> RB6 G
- U10 pad 17: RB7 A -> RB7 G
Routing:
- net +5v: track 191.5 -> 561.5 mm, vias 1 -> 9
- net GND: track 308.7 -> 654.5 mm, vias 0 -> 3
- net I2Cclk: track 8.00 -> 318.0 mm, vias 0 -> 7
- net I2Cdat: track 8.05 -> 307.7 mm, vias 0 -> 8
- net Earth_GND: track 61.6 -> 176.2 mm
- net RB6 G: track 0.00 -> 60.0 mm
- net RB7 G: track 0.00 -> 55.6 mm
- net Net-(U3-RE2/AN7/PSMC3A): track 0.00 -> 48.8 mm, vias 0 -> 1
- net MSCLR E: track 9.52 -> 58.3 mm, vias 0 -> 2
- net C3: track 0.00 -> 46.7 mm
- net Net-(U3-RE1/AN6/PSMC3B): track 0.00 -> 44.9 mm
- net B2: track 0.00 -> 43.5 mm
- net Net-(U3-RA5/AN4/C2OUT/OPA1IN+): track 0.00 -> 39.0 mm
- net Net-(U3-RD6/PSMC3D): track 0.00 -> 38.8 mm, vias 0 -> 1
- net Net-(U3-RA4/C1OUT/OPA1IN+/T0CKI): track 0.00 -> 32.7 mm
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- added copper zone on B.Cu, net GND
Other:
- board size 161.9 x 116.8 mm -> 171.5 x 114.3 mm
- board text added: "GND"

Commit message: added gerber zip files with motherboard and small breakout
Parts:
- C7, C9: footprint Capacitor_THT:CP_Radial_D12.5mm_P2.50mm -> Capacitor_THT:CP_Radial_D6.3mm_P2.50mm
Other:
- board text added: "C_GND"
- board text added: "Midi Bass Guitar Motherboard Rev. A Designed by: Owen Fujii 03/13/2004"

Commit message: updated motherboard pcb
Parts:
- J11: footprint Connector_PinHeader_2.54mm:PinHeader_1x21_P2.54mm_Vertical -> OF Footprints:PinHeader_2x21_P2.54mm_Vertical
Routing:
- net RB6 A: track 60.7 -> 65.2 mm
- net RB7 A: track 55.9 -> 60.0 mm
- net GND: track 654.5 -> 657.0 mm
- net Net-(U8-RD3/PSMC4A): track 39.8 -> 42.0 mm
- net Net-(U8-RD5/PSMC3E): track 56.0 -> 57.5 mm
- net Net-(U8-RD4/PSM3F): track 52.3 -> 53.8 mm
