File: Midi Bass Sch/PowerIn.kicad_sch (KiCad schematic)
At the start: 9 parts

Commit message: working on troubleshooting section of report
Parts:
- J9: renamed from J?; value ? -> Power In
- gave numbers to parts that had none: 8
Changed lines of the file:
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@@
 		(dnp no)
 		(fields_autoplaced yes)
-		(property "Reference" "TP?"
+		(property "Reference" "TP11"
 			(at 153.67 74.1679 0)
 			(effects
@@
 			(project ""
 				(path "/06818073-fb22-48ee-acc5-6dedd827034e/b03edaf9-bff0-4d7c-9ae3-3086f8e495f2"
-					(reference "TP?")
+					(reference "TP11")
 					(unit 1)
 				)
@@
 		(dnp no)
 		(fields_autoplaced yes)
-		(property "Reference" "TP?"
+		(property "Reference" "TP10"
 			(at 95.25 74.1679 0)
 			(effects
@@
 			(project ""
 				(path "/06818073-fb22-48ee-acc5-6dedd827034e/b03edaf9-bff0-4d7c-9ae3-3086f8e495f2"
-					(reference "TP?")
+					(reference "TP10")
 					(unit 1)
 				)
@@
 		(dnp no)
 		(fields_autoplaced yes)
-		(property "Reference" "#PWR0347"
+		(property "Reference" "#PWR0346"
 			(at 148.2344 73.7616 0)
 			(effects
@@
 			(project ""
 				(path "/06818073-fb22-48ee-acc5-6dedd827034e/b03edaf9-bff0-4d7c-9ae3-3086f8e495f2"
-					(reference "#PWR0347")
+					(reference "#PWR0346")
 					(unit 1)
 				)
@@
 		(dnp no)
 		(fields_autoplaced yes)
-		(property "Reference" "L?"
+		(property "Reference" "L93"
 			(at 132.08 73.66 90)
 			(effects
@@
 			(project ""
 				(path "/06818073-fb22-48ee-acc5-6dedd827034e/b03edaf9-bff0-4d7c-9ae3-3086f8e495f2"
-					(reference "L?")
+					(reference "L93")
 					(unit 1)
 				)
@@
 		(dnp no)
 		(fields_autoplaced yes)
-		(property "Reference" "#PWR0345"
+		(property "Reference" "#PWR0347"
 			(at 146.05 88.9 0)
 			(effects
@@
 			(project ""
 				(path "/06818073-fb22-48ee-acc5-6dedd827034e/b03edaf9-bff0-4d7c-9ae3-3086f8e495f2"
-					(reference "#PWR0345")
+					(reference "#PWR0347")
 					(unit 1)
 				)
@@
 		(dnp no)
 		(fields_autoplaced yes)
-		(property "Reference" "C?"
+		(property "Reference" "C8"
 			(at 101.6 81.9149 0)
 			(effects
@@
 			(project ""
 				(path "/06818073-fb22-48ee-acc5-6dedd827034e/b03edaf9-bff0-4d7c-9ae3-3086f8e495f2"
-					(reference "C?")
+					(reference "C8")
 					(unit 1)
 				)
@@
 		(dnp no)
 		(fields_autoplaced yes)
-		(property "Reference" "C?"
+		(property "Reference" "C10"
 			(at 153.67 83.1849 0)
 			(effects
@@
 			(project "Midi Bass Sch"
 				(path "/06818073-fb22-48ee-acc5-6dedd827034e/b03edaf9-bff0-4d7c-9ae3-3086f8e495f2"
-					(reference "C?")
+					(reference "C10")
 					(unit 1)
 				)
@@
 		(dnp no)
 		(fields_autoplaced yes)
-		(property "Reference" "C?"
+		(property "Reference" "C9"
 			(at 142.24 83.1214 0)
 			(effects
@@
 			(project "Midi Bass Sch"
 				(path "/06818073-fb22-48ee-acc5-6dedd827034e/b03edaf9-bff0-4d7c-9ae3-3086f8e495f2"
-					(reference "C?")
+					(reference "C9")
 					(unit 1)
 				)
@@
 		(dnp no)
 		(fields_autoplaced yes)
-		(property "Reference" "J?"
+		(property "Reference" "J9"
 			(at 72.39 71.12 0)
 			(effects
@@
 			)
 		)
-		(property "Value" "?"
+		(property "Value" "Power In"
 			(at 72.39 73.66 0)
 			(effects
@@
 			(project ""
 				(path "/06818073-fb22-48ee-acc5-6dedd827034e/b03edaf9-bff0-4d7c-9ae3-3086f8e495f2"
-					(reference "J?")
+					(reference "J9")
 					(unit 1)
 				)
@@
 		(dnp no)
 		(fields_autoplaced yes)
-		(property "Reference" "U?"
+		(property "Reference" "U31"
 			(at 118.11 72.39 0)
 			(effects
@@
 			(project ""
 				(path "/06818073-fb22-48ee-acc5-6dedd827034e/b03edaf9-bff0-4d7c-9ae3-3086f8e495f2"
-					(reference "U?")
+					(reference "U31")
 					(unit 1)
 				)
@@
 		(dnp no)
 		(fields_autoplaced yes)
-		(property "Reference" "#PWR0344"
+		(property "Reference" "#PWR0345"
 			(at 93.98 88.9 0)
 			(effects
@@
 			(project ""
 				(path "/06818073-fb22-48ee-acc5-6dedd827034e/b03edaf9-bff0-4d7c-9ae3-3086f8e495f2"
-					(reference "#PWR0344")
+					(reference "#PWR0345")
 					(unit 1)
 				)
@@
 		(dnp no)
 		(fields_autoplaced yes)
-		(property "Reference" "C?"
+		(property "Reference" "C7"
 			(at 90.17 81.8514 0)
 			(effects
@@
 			(project ""
 				(path "/06818073-fb22-48ee-acc5-6dedd827034e/b03edaf9-bff0-4d7c-9ae3-3086f8e495f2"
-					(reference "C?")
+					(reference "C7")
 					(unit 1)
 				)
@@
 		(dnp no)
 		(fields_autoplaced yes)
-		(property "Reference" "#PWR0346"
+		(property "Reference" "#PWR0344"
 			(at 87.2744 73.7616 0)
 			(effects
@@
 			(project ""
 				(path "/06818073-fb22-48ee-acc5-6dedd827034e/b03edaf9-bff0-4d7c-9ae3-3086f8e495f2"
-					(reference "#PWR0346")
-					(unit 1)
-				)
+					(reference "#PWR0344")
+					(unit 1)
+				)

Commit message: working on final troubleshooting sections, modified pluck slave to header connections
Parts:
- renumbered J9 to J11
Changed lines of the file:
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@@
 		(dnp no)
 		(fields_autoplaced yes)
-		(property "Reference" "#PWR0346"
+		(property "Reference" "#PWR0348"
 			(at 148.2344 73.7616 0)
 			(effects
@@
 			(project ""
 				(path "/06818073-fb22-48ee-acc5-6dedd827034e/b03edaf9-bff0-4d7c-9ae3-3086f8e495f2"
-					(reference "#PWR0346")
+					(reference "#PWR0348")
 					(unit 1)
 				)
@@
 		(dnp no)
 		(fields_autoplaced yes)
-		(property "Reference" "#PWR0347"
+		(property "Reference" "#PWR0349"
 			(at 146.05 88.9 0)
 			(effects
@@
 			(project ""
 				(path "/06818073-fb22-48ee-acc5-6dedd827034e/b03edaf9-bff0-4d7c-9ae3-3086f8e495f2"
-					(reference "#PWR0347")
+					(reference "#PWR0349")
 					(unit 1)
 				)
@@
 		(dnp no)
 		(fields_autoplaced yes)
-		(property "Reference" "J9"
+		(property "Reference" "J11"
 			(at 72.39 71.12 0)
 			(effects
@@
 			(project ""
 				(path "/06818073-fb22-48ee-acc5-6dedd827034e/b03edaf9-bff0-4d7c-9ae3-3086f8e495f2"
-					(reference "J9")
+					(reference "J11")
 					(unit 1)
 				)
@@
 		(dnp no)
 		(fields_autoplaced yes)
-		(property "Reference" "#PWR0345"
+		(property "Reference" "#PWR0347"
 			(at 93.98 88.9 0)
 			(effects
@@
 			(project ""
 				(path "/06818073-fb22-48ee-acc5-6dedd827034e/b03edaf9-bff0-4d7c-9ae3-3086f8e495f2"
-					(reference "#PWR0345")
+					(reference "#PWR0347")
 					(unit 1)
 				)
@@
 		(dnp no)
 		(fields_autoplaced yes)
-		(property "Reference" "#PWR0344"
+		(property "Reference" "#PWR0346"
 			(at 87.2744 73.7616 0)
 			(effects
@@
 			(project ""
 				(path "/06818073-fb22-48ee-acc5-6dedd827034e/b03edaf9-bff0-4d7c-9ae3-3086f8e495f2"
-					(reference "#PWR0344")
-					(unit 1)
-				)
+					(reference "#PWR0346")
+					(unit 1)
+				)

Commit message: finished troubleshooting section
Parts:
- renumbered J11 to J13
Changed lines of the file:
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@@
 		(dnp no)
 		(fields_autoplaced yes)
-		(property "Reference" "#PWR0348"
+		(property "Reference" "#PWR0350"
 			(at 148.2344 73.7616 0)
 			(effects
@@
 			(project ""
 				(path "/06818073-fb22-48ee-acc5-6dedd827034e/b03edaf9-bff0-4d7c-9ae3-3086f8e495f2"
-					(reference "#PWR0348")
+					(reference "#PWR0350")
 					(unit 1)
 				)
@@
 		(dnp no)
 		(fields_autoplaced yes)
-		(property "Reference" "#PWR0349"
+		(property "Reference" "#PWR0351"
 			(at 146.05 88.9 0)
 			(effects
@@
 			(project ""
 				(path "/06818073-fb22-48ee-acc5-6dedd827034e/b03edaf9-bff0-4d7c-9ae3-3086f8e495f2"
-					(reference "#PWR0349")
+					(reference "#PWR0351")
 					(unit 1)
 				)
@@
 		(dnp no)
 		(fields_autoplaced yes)
-		(property "Reference" "J11"
+		(property "Reference" "J13"
 			(at 72.39 71.12 0)
 			(effects
@@
 			(project ""
 				(path "/06818073-fb22-48ee-acc5-6dedd827034e/b03edaf9-bff0-4d7c-9ae3-3086f8e495f2"
-					(reference "J11")
+					(reference "J13")
 					(unit 1)
 				)
@@
 		(dnp no)
 		(fields_autoplaced yes)
-		(property "Reference" "#PWR0347"
+		(property "Reference" "#PWR0349"
 			(at 93.98 88.9 0)
 			(effects
@@
 			(project ""
 				(path "/06818073-fb22-48ee-acc5-6dedd827034e/b03edaf9-bff0-4d7c-9ae3-3086f8e495f2"
-					(reference "#PWR0347")
+					(reference "#PWR0349")
 					(unit 1)
 				)
@@
 		(dnp no)
 		(fields_autoplaced yes)
-		(property "Reference" "#PWR0346"
+		(property "Reference" "#PWR0348"
 			(at 87.2744 73.7616 0)
 			(effects
@@
 			(project ""
 				(path "/06818073-fb22-48ee-acc5-6dedd827034e/b03edaf9-bff0-4d7c-9ae3-3086f8e495f2"
-					(reference "#PWR0346")
-					(unit 1)
-				)
+					(reference "#PWR0348")
+					(unit 1)
+				)

Commit message: began getting images for schematic appendix
Other:
- title: (none) -> Input Power Schematic
Changed lines of the file:
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@@
 	(generator_version "8.0")
 	(paper "A")
+	(title_block
+		(title "Input Power Schematic")
+		(date "2024-12-10")
+		(rev "A")
+	)
 	(junction
 		(at 92.71 78.74)

Commit message: began working on pcb layout deleted extra schematics for solenoid break out board
Parts:
- C10, C8: footprint (none) -> Capacitor_SMD:C_0805_2012Metric_Pad1.18x1.45mm_HandSolder
- C7, C9: footprint (none) -> Capacitor_THT:CP_Radial_D12.5mm_P2.50mm
- J16: renamed from J13; footprint (none) -> OF footprints:Two_Pin_Screw_Terminal
- L33: renamed from L93; footprint (none) -> Inductor_THT:L_Axial_L5.0mm_D3.6mm_P10.00mm_Horizontal_Murata_BL01RN1A2A2
- TP10, TP11: footprint (none) -> Connector_PinHeader_2.54mm:PinHeader_1x01_P2.54mm_Vertical
- renumbered U31 to U16
Changed lines of the file:
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@@
 			)
 		)
-		(property "Footprint" ""
+		(property "Footprint" "Connector_PinHeader_2.54mm:PinHeader_1x01_P2.54mm_Vertical"
 			(at 156.21 78.74 0)
 			(effects
@@
 			)
 		)
-		(property "Footprint" ""
+		(property "Footprint" "Connector_PinHeader_2.54mm:PinHeader_1x01_P2.54mm_Vertical"
 			(at 97.79 78.74 0)
 			(effects
@@
 		(dnp no)
 		(fields_autoplaced yes)
-		(property "Reference" "#PWR0350"
+		(property "Reference" "#PWR0173"
 			(at 148.2344 73.7616 0)
 			(effects
@@
 			(project ""
 				(path "/06818073-fb22-48ee-acc5-6dedd827034e/b03edaf9-bff0-4d7c-9ae3-3086f8e495f2"
-					(reference "#PWR0350")
+					(reference "#PWR0173")
 					(unit 1)
 				)
@@
 		(dnp no)
 		(fields_autoplaced yes)
-		(property "Reference" "L93"
+		(property "Reference" "L33"
 			(at 132.08 73.66 90)
 			(effects
@@
 			)
 		)
-		(property "Footprint" ""
+		(property "Footprint" "Inductor_THT:L_Axial_L5.0mm_D3.6mm_P10.00mm_Horizontal_Murata_BL01RN1A2A2"
 			(at 132.08 78.74 0)
 			(effects
@@
 			(project ""
 				(path "/06818073-fb22-48ee-acc5-6dedd827034e/b03edaf9-bff0-4d7c-9ae3-3086f8e495f2"
-					(reference "L93")
+					(reference "L33")
 					(unit 1)
 				)
@@
 		(dnp no)
 		(fields_autoplaced yes)
-		(property "Reference" "#PWR0351"
+		(property "Reference" "#PWR0174"
 			(at 146.05 88.9 0)
 			(effects
@@
 			(project ""
 				(path "/06818073-fb22-48ee-acc5-6dedd827034e/b03edaf9-bff0-4d7c-9ae3-3086f8e495f2"
-					(reference "#PWR0351")
+					(reference "#PWR0174")
 					(unit 1)
 				)
@@
 			)
 		)
-		(property "Footprint" ""
+		(property "Footprint" "Capacitor_SMD:C_0805_2012Metric_Pad1.18x1.45mm_HandSolder"
 			(at 99.06 77.47 0)
 			(effects
@@
 			)
 		)
-		(property "Footprint" ""
+		(property "Footprint" "Capacitor_SMD:C_0805_2012Metric_Pad1.18x1.45mm_HandSolder"
 			(at 151.13 78.74 0)
 			(effects
@@
 			)
 		)
-		(property "Footprint" ""
+		(property "Footprint" "Capacitor_THT:CP_Radial_D12.5mm_P2.50mm"
 			(at 139.7 78.74 0)
 			(effects
@@
 		(dnp no)
 		(fields_autoplaced yes)
-		(property "Reference" "J13"
+		(property "Reference" "J16"
 			(at 72.39 71.12 0)
 			(effects
@@
 			)
 		)
-		(property "Footprint" ""
+		(property "Footprint" "OF footprints:Two_Pin_Screw_Terminal"
 			(at 72.39 74.93 0)
 			(effects
@@
 			(project ""
 				(path "/06818073-fb22-48ee-acc5-6dedd827034e/b03edaf9-bff0-4d7c-9ae3-3086f8e495f2"
-					(reference "J13")
+					(reference "J16")
 					(unit 1)
 				)
@@
 		(dnp no)
 		(fields_autoplaced yes)
-		(property "Reference" "U31"
+		(property "Reference" "U16"
 			(at 118.11 72.39 0)
 			(effects
@@
 			(project ""
 				(path "/06818073-fb22-48ee-acc5-6dedd827034e/b03edaf9-bff0-4d7c-9ae3-3086f8e495f2"
-					(reference "U31")
+					(reference "U16")
 					(unit 1)
 				)
@@
 		(dnp no)
 		(fields_autoplaced yes)
-		(property "Reference" "#PWR0349"
+		(property "Reference" "#PWR0172"
 			(at 93.98 88.9 0)
 			(effects
@@
 			(project ""
 				(path "/06818073-fb22-48ee-acc5-6dedd827034e/b03edaf9-bff0-4d7c-9ae3-3086f8e495f2"
-					(reference "#PWR0349")
+					(reference "#PWR0172")
 					(unit 1)
 				)
@@
 			)
 		)
-		(property "Footprint" ""
+		(property "Footprint" "Capacitor_THT:CP_Radial_D12.5mm_P2.50mm"
 			(at 87.63 77.47 0)
 			(effects
@@
 		(dnp no)
 		(fields_autoplaced yes)
-		(property "Reference" "#PWR0348"
+		(property "Reference" "#PWR0171"
 			(at 87.2744 73.7616 0)
 			(effects
@@
 			(project ""
 				(path "/06818073-fb22-48ee-acc5-6dedd827034e/b03edaf9-bff0-4d7c-9ae3-3086f8e495f2"
-					(reference "#PWR0348")
-					(unit 1)
-				)
+					(reference "#PWR0171")
+					(unit 1)
+				)

Commit message: created pcb for breakout working on pcb for main control board
Changed lines of the file:
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@@
 (kicad_sch
-	(version 20231120)
+	(version 20250114)
 	(generator "eeschema")
-	(generator_version "8.0")
+	(generator_version "9.0")
 	(paper "A")
 	(title_block

Commit message: updated motherboard pcb
Parts:
- C7, C9: footprint Capacitor_THT:CP_Radial_D12.5mm_P2.50mm -> Capacitor_THT:CP_Radial_D6.3mm_P2.50mm
Changed lines of the file:
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@@
 			)
 		)
-		(property "Footprint" "Capacitor_THT:CP_Radial_D12.5mm_P2.50mm"
+		(property "Footprint" "Capacitor_THT:CP_Radial_D6.3mm_P2.50mm"
 			(at 139.7 78.74 0)
 			(effects
@@
 			)
 		)
-		(property "Footprint" "Capacitor_THT:CP_Radial_D12.5mm_P2.50mm"
+		(property "Footprint" "Capacitor_THT:CP_Radial_D6.3mm_P2.50mm"
 			(at 87.63 77.47 0)
 			(effects

Commit message: created and generated Rev. B of Motherboard
Parts:
- renumbered C7 to C4, C8 to C5, C9 to C6, C10 to C7, J16 to J9, L33 to L1, TP10 to TP7, TP11 to TP8, U16 to U4
Changed lines of the file:
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@@
 		(dnp no)
 		(fields_autoplaced yes)
-		(property "Reference" "TP11"
+		(property "Reference" "TP8"
 			(at 153.67 74.1679 0)
 			(effects
@@
 			(project ""
 				(path "/06818073-fb22-48ee-acc5-6dedd827034e/b03edaf9-bff0-4d7c-9ae3-3086f8e495f2"
-					(reference "TP11")
+					(reference "TP8")
 					(unit 1)
 				)
@@
 		(dnp no)
 		(fields_autoplaced yes)
-		(property "Reference" "TP10"
+		(property "Reference" "TP7"
 			(at 95.25 74.1679 0)
 			(effects
@@
 			(project ""
 				(path "/06818073-fb22-48ee-acc5-6dedd827034e/b03edaf9-bff0-4d7c-9ae3-3086f8e495f2"
-					(reference "TP10")
+					(reference "TP7")
 					(unit 1)
 				)
@@
 		(dnp no)
 		(fields_autoplaced yes)
-		(property "Reference" "#PWR0173"
+		(property "Reference" "#PWR047"
 			(at 148.2344 73.7616 0)
 			(effects
@@
 			(project ""
 				(path "/06818073-fb22-48ee-acc5-6dedd827034e/b03edaf9-bff0-4d7c-9ae3-3086f8e495f2"
-					(reference "#PWR0173")
+					(reference "#PWR047")
 					(unit 1)
 				)
@@
 		(dnp no)
 		(fields_autoplaced yes)
-		(property "Reference" "L33"
+		(property "Reference" "L1"
 			(at 132.08 73.66 90)
 			(effects
@@
 			(project ""
 				(path "/06818073-fb22-48ee-acc5-6dedd827034e/b03edaf9-bff0-4d7c-9ae3-3086f8e495f2"
-					(reference "L33")
+					(reference "L1")
 					(unit 1)
 				)
@@
 		(dnp no)
 		(fields_autoplaced yes)
-		(property "Reference" "#PWR0174"
+		(property "Reference" "#PWR048"
 			(at 146.05 88.9 0)
 			(effects
@@
 			(project ""
 				(path "/06818073-fb22-48ee-acc5-6dedd827034e/b03edaf9-bff0-4d7c-9ae3-3086f8e495f2"
-					(reference "#PWR0174")
+					(reference "#PWR048")
 					(unit 1)
 				)
@@
 		(dnp no)
 		(fields_autoplaced yes)
-		(property "Reference" "C8"
+		(property "Reference" "C5"
 			(at 101.6 81.9149 0)
 			(effects
@@
 			(project ""
 				(path "/06818073-fb22-48ee-acc5-6dedd827034e/b03edaf9-bff0-4d7c-9ae3-3086f8e495f2"
-					(reference "C8")
+					(reference "C5")
 					(unit 1)
 				)
@@
 		(dnp no)
 		(fields_autoplaced yes)
-		(property "Reference" "C10"
+		(property "Reference" "C7"
 			(at 153.67 83.1849 0)
 			(effects
@@
 			(project "Midi Bass Sch"
 				(path "/06818073-fb22-48ee-acc5-6dedd827034e/b03edaf9-bff0-4d7c-9ae3-3086f8e495f2"
-					(reference "C10")
+					(reference "C7")
 					(unit 1)
 				)
@@
 		(dnp no)
 		(fields_autoplaced yes)
-		(property "Reference" "C9"
+		(property "Reference" "C6"
 			(at 142.24 83.1214 0)
 			(effects
@@
 			(project "Midi Bass Sch"
 				(path "/06818073-fb22-48ee-acc5-6dedd827034e/b03edaf9-bff0-4d7c-9ae3-3086f8e495f2"
-					(reference "C9")
+					(reference "C6")
 					(unit 1)
 				)
@@
 		(dnp no)
 		(fields_autoplaced yes)
-		(property "Reference" "J16"
+		(property "Reference" "J9"
 			(at 72.39 71.12 0)
 			(effects
@@
 			(project ""
 				(path "/06818073-fb22-48ee-acc5-6dedd827034e/b03edaf9-bff0-4d7c-9ae3-3086f8e495f2"
-					(reference "J16")
+					(reference "J9")
 					(unit 1)
 				)
@@
 		(dnp no)
 		(fields_autoplaced yes)
-		(property "Reference" "U16"
+		(property "Reference" "U4"
 			(at 118.11 72.39 0)
 			(effects
@@
 			(project ""
 				(path "/06818073-fb22-48ee-acc5-6dedd827034e/b03edaf9-bff0-4d7c-9ae3-3086f8e495f2"
-					(reference "U16")
+					(reference "U4")
 					(unit 1)
 				)
@@
 		(dnp no)
 		(fields_autoplaced yes)
-		(property "Reference" "#PWR0172"
+		(property "Reference" "#PWR046"
 			(at 93.98 88.9 0)
 			(effects
@@
 			(project ""
 				(path "/06818073-fb22-48ee-acc5-6dedd827034e/b03edaf9-bff0-4d7c-9ae3-3086f8e495f2"
-					(reference "#PWR0172")
+					(reference "#PWR046")
 					(unit 1)
 				)
@@
 		(dnp no)
 		(fields_autoplaced yes)
-		(property "Reference" "C7"
+		(property "Reference" "C4"
 			(at 90.17 81.8514 0)
 			(effects
@@
 			(project ""
 				(path "/06818073-fb22-48ee-acc5-6dedd827034e/b03edaf9-bff0-4d7c-9ae3-3086f8e495f2"
-					(reference "C7")
+					(reference "C4")
 					(unit 1)
 				)
@@
 		(dnp no)
 		(fields_autoplaced yes)
-		(property "Reference" "#PWR0171"
+		(property "Reference" "#PWR045"
 			(at 87.2744 73.7616 0)
 			(effects
@@
 			(project ""
 				(path "/06818073-fb22-48ee-acc5-6dedd827034e/b03edaf9-bff0-4d7c-9ae3-3086f8e495f2"
-					(reference "#PWR0171")
-					(unit 1)
-				)
+					(reference "#PWR045")
+					(unit 1)
+				)
