File: Small Unit Breakout/Small Unit Breakout.kicad_pcb (KiCad board)
At the start: 2 copper layers, 65 parts, among them J1 Power In, J2 Pluck IN, Q1 STN851-A, Q10 STN851-A, Q11 STN851-A, Q12 STN851-A, Q2 STN851-A, Q3 STN851-A, Q4 STN851-A, Q5 STN851-A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

Commit message: added gerber zip files with motherboard and small breakout
Parts:
- added ?: , , F.Cu at (109.2, 67.9)
- added ?: , , F.Cu at (109.2, 136.5)
- added ?: , , F.Cu at (45.1, 136.5)
- added G***: LOGO, Logos:Wisteria Logo .5x.5, F.Cu at (108.0, 108.6)
- added G***: LOGO, Logos:ISU 1inch, F.Cu at (56.5, 134.6)
- added Power: Two_Pin_Screw_Terminal, OF Footprints:Two_Pin_Screw_Terminal, F.Cu at (108.6, 124.5)
- added REF**: 6-32 Mount, OF Footprints:6-32 Mount, F.Cu at (45.1, 67.9)
- moved J1 102.3 mm to (45.7, 77.5), turned to -90 degrees
- moved Q10 84.6 mm to (92.1, 136.5)
- moved D10 74.4 mm to (69.5, 117.5)
- moved D9 73.8 mm to (69.5, 113.7)
- moved D8 70.3 mm to (69.5, 106.0)
- moved D7 69.7 mm to (69.5, 102.2)
- moved D11 66.4 mm to (69.5, 109.9)
- moved D12 65.7 mm to (69.5, 121.3)
- moved D1 63.7 mm to (69.5, 98.4)
- moved Q9 62.4 mm to (83.2, 130.8)
- moved Q11 61.8 mm to (83.2, 119.4)
- moved D2 58.6 mm to (69.5, 94.6)
- moved Q12 56.9 mm to (92.1, 125.1)
- moved Q7 56.3 mm to (83.2, 108.0)
- moved Q8 52.7 mm to (92.1, 113.7)
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Routing:
- net +12v: track 5.26 -> 243.0 mm
- net Net-(Q10-B): track 0.00 -> 25.8 mm
- net Net-(Q12-B): track 0.00 -> 22.9 mm
- net Net-(Q4-B): track 0.00 -> 20.8 mm
- net Net-(Q8-B): track 0.00 -> 18.9 mm
- net Net-(Q6-B): track 0.00 -> 18.8 mm
- net Net-(Q2-B): track 0.00 -> 17.4 mm
- net Net-(R7-Pad1): track 0.00 -> 13.9 mm
- net Net-(D3-K): track 0.00 -> 13.8 mm
- net Net-(Q3-B): track 0.00 -> 13.3 mm
- net Net-(R22-Pad1): track 0.00 -> 13.2 mm
- net Net-(Q9-B): track 0.00 -> 12.6 mm
- net Net-(R21-Pad1): track 0.00 -> 12.5 mm
- net Net-(R8-Pad1): track 0.00 -> 12.5 mm
- net Net-(R24-Pad1): track 0.00 -> 12.0 mm
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- added copper zone on B.Cu, net Chassis_GND
Other:
- board outline added: 71.8 x 76.2 mm
- board text added: "+"
- board text added: "Pluck Breakout Rev. A Designed By: Owen Fujii 03/13/2025"
