File: Solenoid Breakout Board/Solenoid Breakout Board.kicad_pcb (KiCad board)
At the start: 2 copper layers, 106 parts, among them J1 Solenoid In, Q1 STN851-A, Q10 STN851-A, Q11 STN851-A, Q12 STN851-A, Q13 STN851-A, Q14 STN851-A, Q15 STN851-A, Q16 STN851-A, Q17 STN851-A, Q18 STN851-A, Q19 STN851-A, Q2 STN851-A, Q20 STN851-A, Q3 STN851-A, Q4 STN851-A, Q5 STN851-A, Q6 STN851-A, Q7 STN851-A, Q8 STN851-A, Q9 STN851-A, U1 LTV-247, U2 LTV-247, U3 LTV-247, U4 LTV-247, U5 LTV-247

Commit message: finished rev A pcb for breakout:
Parts:
- added G***: LOGO, Logos:ISU 1inch, F.Cu at (163.2, 134.0)
- added G***: LOGO, Logos:Bengal Head .5x.5, F.Cu at (51.4, 140.3)
- added G***: LOGO, Logos:Wisteria Logo .75x.75, F.Cu at (64.8, 142.9)
- added POWER: Two_Pin_Screw_Terminal, OF footprints:Two_Pin_Screw_Terminal, F.Cu at (175.9, 127.0)
- added POWER: Two_Pin_Screw_Terminal, OF footprints:Two_Pin_Screw_Terminal, F.Cu at (48.9, 127.0)
- added Power Out: Pwr IN, Connector_PinHeader_2.54mm:PinHeader_1x02_P2.54mm_Vertical, F.Cu at (47.0, 98.4)
- added REF**: 6-32 Mount, OF footprints:6-32 Mount, F.Cu at (176.5, 91.4)
- added REF**: 6-32 Mount, OF footprints:6-32 Mount, F.Cu at (48.3, 91.4)
- added REF**: 6-32 Mount, OF footprints:6-32 Mount, F.Cu at (176.5, 151.8)
- added REF**: 6-32 Mount, OF footprints:6-32 Mount, F.Cu at (48.3, 151.8)
- moved L20 101.1 mm to (173.4, 98.4)
- moved L19 98.7 mm to (167.0, 108.0)
- moved L18 97.7 mm to (160.7, 98.4)
- moved L17 95.3 mm to (154.3, 108.0)
- moved L16 94.3 mm to (148.0, 98.4)
- moved Q17 92.9 mm to (154.3, 117.5), turned to 90 degrees
- moved Q19 90.1 mm to (167.0, 117.5), turned to 90 degrees
- moved Q20 85.9 mm to (173.4, 108.0), turned to 90 degrees
- moved Q18 84.4 mm to (160.7, 107.9), turned to 90 degrees
- moved Q13 83.9 mm to (128.7, 117.5), turned to 90 degrees
- moved Q15 78.5 mm to (141.6, 117.5), turned to 90 degrees
- moved Q9 77.8 mm to (122.3, 108.0), turned to 90 degrees
- moved Q14 73.1 mm to (135.0, 108.0), turned to 90 degrees
- moved Q16 72.3 mm to (148.0, 108.0), turned to 90 degrees
- moved L15 68.9 mm to (141.6, 108.0)
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Routing:
- net +12v: track 0.00 -> 416.3 mm
- net GND: track 0.00 -> 59.0 mm
- net Net-(D6-K): track 0.00 -> 31.2 mm
- net Net-(R8-Pad1): track 0.00 -> 31.0 mm
- net Net-(R40-Pad1): track 0.00 -> 28.3 mm
- net Net-(D2-K): track 0.00 -> 28.2 mm
- net Net-(R7-Pad1): track 0.00 -> 28.1 mm
- net Net-(D20-K): track 0.00 -> 26.6 mm
- net Net-(R39-Pad1): track 0.00 -> 26.4 mm
- net Net-(D3-K): track 0.00 -> 25.2 mm
- net Net-(R10-Pad1): track 0.00 -> 25.0 mm
- net Net-(Q20-B): track 0.00 -> 24.9 mm
- net Net-(D19-K): track 0.00 -> 24.1 mm
- net Net-(R38-Pad1): track 0.00 -> 23.5 mm
- net Net-(Q18-B): track 0.00 -> 22.9 mm
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- added copper zone on B.Cu, net Chassis_GND
Other:
- board outline added: 135.9 x 67.9 mm
- board text added: "+"
- board text added: "GND"
- board text added: "Solenoid Breakout Board Rev. A Designed By: Owen Fujii 03/10/2025"

Commit message: revised schematic for breakout updating PCB to match
Parts:
- removed the D1 at (83.8, 127.0)
- removed the L1 at (58.8, 98.4)
- removed POWER (x2): Two_Pin_Screw_Terminal, OF footprints:Two_Pin_Screw_Terminal
- removed the R13 at (106.7, 148.5)
- removed the R14 at (109.2, 148.5)
- removed the R15 at (111.8, 148.5)
- removed the R22 at (91.4, 125.7)
- removed the R23 at (96.5, 125.7)
- removed REF** (x4): 6-32 Mount, OF footprints:6-32 Mount
- added D21: LED, LED_SMD:LED_0805_2012Metric_Pad1.15x1.40mm_HandSolder, F.Cu at (-90.0, 150.2)
- added D22: LED, LED_SMD:LED_0805_2012Metric_Pad1.15x1.40mm_HandSolder, F.Cu at (-90.0, 153.3)
- added D23: 1N4148, LED_SMD:LED_0805_2012Metric_Pad1.15x1.40mm_HandSolder, F.Cu at (-101.6, 144.4)
- added D24: 1N4148, LED_SMD:LED_0805_2012Metric_Pad1.15x1.40mm_HandSolder, F.Cu at (-101.6, 147.9)
- added D25: 1N4148, LED_SMD:LED_0805_2012Metric_Pad1.15x1.40mm_HandSolder, F.Cu at (-101.6, 151.5)
- added D26: 1N4148, LED_SMD:LED_0805_2012Metric_Pad1.15x1.40mm_HandSolder, F.Cu at (-101.6, 155.0)
- added D27: LED, LED_SMD:LED_0805_2012Metric_Pad1.15x1.40mm_HandSolder, F.Cu at (-90.0, 156.3)
- added D28: LED, LED_SMD:LED_0805_2012Metric_Pad1.15x1.40mm_HandSolder, F.Cu at (-90.0, 159.3)
- added D29: LED, LED_SMD:LED_0805_2012Metric_Pad1.15x1.40mm_HandSolder, F.Cu at (-85.2, 144.1)
- added D30: LED, LED_SMD:LED_0805_2012Metric_Pad1.15x1.40mm_HandSolder, F.Cu at (-85.2, 147.2)
- added D31: 1N4148, LED_SMD:LED_0805_2012Metric_Pad1.15x1.40mm_HandSolder, F.Cu at (-101.6, 158.6)
- added D32: 1N4148, LED_SMD:LED_0805_2012Metric_Pad1.15x1.40mm_HandSolder, F.Cu at (-101.6, 162.1)
- added D33: 1N4148, LED_SMD:LED_0805_2012Metric_Pad1.15x1.40mm_HandSolder, F.Cu at (-101.6, 165.7)
- added D34: 1N4148, LED_SMD:LED_0805_2012Metric_Pad1.15x1.40mm_HandSolder, F.Cu at (-101.6, 169.2)
- added D35: LED, LED_SMD:LED_0805_2012Metric_Pad1.15x1.40mm_HandSolder, F.Cu at (-85.2, 150.2)
- added D36: LED, LED_SMD:LED_0805_2012Metric_Pad1.15x1.40mm_HandSolder, F.Cu at (-85.2, 153.3)
- added D37: LED, LED_SMD:LED_0805_2012Metric_Pad1.15x1.40mm_HandSolder, F.Cu at (-85.2, 156.3)
- added D38: 1N4148, LED_SMD:LED_0805_2012Metric_Pad1.15x1.40mm_HandSolder, F.Cu at (-101.6, 172.8)
- added D39: 1N4148, LED_SMD:LED_0805_2012Metric_Pad1.15x1.40mm_HandSolder, F.Cu at (-101.6, 176.3)
- added D40: 1N4148, LED_SMD:LED_0805_2012Metric_Pad1.15x1.40mm_HandSolder, F.Cu at (-101.6, 179.9)
- added D6: 1N4148, LED_SMD:LED_0805_2012Metric_Pad1.15x1.40mm_HandSolder, F.Cu at (-101.6, 34.2)
- added J3: Pwr OUT, OF Footprints:Two_Pin_Screw_Terminal, F.Cu at (-85.3, 43.2)
- added L2: Solenoid, OF Footprints:Small Expanded TH, F.Cu at (-105.3, 6.76)
- added R16: 1kΩ, Resistor_SMD:R_0805_2012Metric_Pad1.20x1.40mm_HandSolder, F.Cu at (-87.4, 66.9)
- added R17: 1kΩ, Resistor_SMD:R_0805_2012Metric_Pad1.20x1.40mm_HandSolder, F.Cu at (-87.4, 69.9)
- added R18: 1kΩ, Resistor_SMD:R_0805_2012Metric_Pad1.20x1.40mm_HandSolder, F.Cu at (-87.4, 72.8)
- added R41: 1kΩ, Resistor_SMD:R_0805_2012Metric_Pad1.20x1.40mm_HandSolder, F.Cu at (120.7, 148.3)
- added R42: 1kΩ, Resistor_SMD:R_0805_2012Metric_Pad1.20x1.40mm_HandSolder, F.Cu at (123.2, 148.3)
- added R43: 1kΩ, Resistor_SMD:R_0805_2012Metric_Pad1.20x1.40mm_HandSolder, F.Cu at (118.1, 148.3)
- added R44: 1kΩ, Resistor_SMD:R_0805_2012Metric_Pad1.20x1.40mm_HandSolder, F.Cu at (-54.9, 134.7)
- added R45: 1kΩ, Resistor_SMD:R_0805_2012Metric_Pad1.20x1.40mm_HandSolder, F.Cu at (-54.9, 137.6)
- added R46: 1kΩ, Resistor_SMD:R_0805_2012Metric_Pad1.20x1.40mm_HandSolder, F.Cu at (-54.9, 140.6)
- added R47: 1kΩ, Resistor_SMD:R_0805_2012Metric_Pad1.20x1.40mm_HandSolder, F.Cu at (-54.9, 143.5)
- added R48: 68Ω, Resistor_SMD:R_0805_2012Metric_Pad1.20x1.40mm_HandSolder, F.Cu at (-22.8, 51.1)
- added R49: 68Ω, Resistor_SMD:R_0805_2012Metric_Pad1.20x1.40mm_HandSolder, F.Cu at (-22.8, 54.0)
- added R50: 68Ω, Resistor_SMD:R_0805_2012Metric_Pad1.20x1.40mm_HandSolder, F.Cu at (-18.1, 39.3)
- added R51: 68Ω, Resistor_SMD:R_0805_2012Metric_Pad1.20x1.40mm_HandSolder, F.Cu at (-18.1, 42.2)
- added R52: 1kΩ, Resistor_SMD:R_0805_2012Metric_Pad1.20x1.40mm_HandSolder, F.Cu at (129.5, 148.3)
- added R53: 1kΩ, Resistor_SMD:R_0805_2012Metric_Pad1.20x1.40mm_HandSolder, F.Cu at (132.1, 148.3)
- added R54: 1kΩ, Resistor_SMD:R_0805_2012Metric_Pad1.20x1.40mm_HandSolder, F.Cu at (134.6, 148.3)
- added R55: 1kΩ, Resistor_SMD:R_0805_2012Metric_Pad1.20x1.40mm_HandSolder, F.Cu at (-50.2, 137.6)
- added R56: 1kΩ, Resistor_SMD:R_0805_2012Metric_Pad1.20x1.40mm_HandSolder, F.Cu at (-50.2, 140.6)
- added R57: 1kΩ, Resistor_SMD:R_0805_2012Metric_Pad1.20x1.40mm_HandSolder, F.Cu at (-50.2, 143.5)
- added R58: 68Ω, Resistor_SMD:R_0805_2012Metric_Pad1.20x1.40mm_HandSolder, F.Cu at (-18.1, 45.2)
- added R59: 68Ω, Resistor_SMD:R_0805_2012Metric_Pad1.20x1.40mm_HandSolder, F.Cu at (-18.1, 48.1)
- added R6: 1kΩ, Resistor_SMD:R_0805_2012Metric_Pad1.20x1.40mm_HandSolder, F.Cu at (66.0, 126.0)
- added R60: 68Ω, Resistor_SMD:R_0805_2012Metric_Pad1.20x1.40mm_HandSolder, F.Cu at (-18.1, 51.1)
- added R8: 1kΩ, Resistor_SMD:R_0805_2012Metric_Pad1.20x1.40mm_HandSolder, F.Cu at (-87.4, 64.0)
- D12, D13, D14, D17, D18, D5, D7, D8: value LED -> 1N4148
- J2: renamed from Power Out; footprint Connector_PinHeader_2.54mm:PinHeader_1x02_P2.54mm_Vertical -> OF Footprints:Two_Pin_Screw_Terminal
- L1: renamed from L2; footprint Connector_PinHeader_2.54mm:PinHeader_1x02_P2.54mm_Vertical -> OF Footprints:Small Expanded TH
- L10, L11, L12, L13, L14, L16, L17, L18, L19, L20, L3, L4, L5, L6, L7, L8, L9: footprint Connector_PinHeader_2.54mm:PinHeader_1x02_P2.54mm_Vertical -> OF Footprints:Small Expanded TH
- L15: footprint Connector_PinHeader_2.54mm:PinHeader_1x02_P2.54mm_Vertical -> OF Footprints:Small Expanded TH; moved to B.Cu
- Q1: value STN851-A -> IRF540N; footprint Package_TO_SOT_SMD:SOT-223-3_TabPin2 -> Package_TO_SOT_THT:TO-220-3_Vertical; moved to B.Cu
- Q10, Q11, Q12, Q13, Q14, Q15, Q16, Q17, Q18, Q19, Q2, Q20, Q3, Q4, Q5, Q6, Q7, Q8, Q9: value STN851-A -> IRF540N; footprint Package_TO_SOT_SMD:SOT-223-3_TabPin2 -> Package_TO_SOT_THT:TO-220-3_Vertical
- R1: renamed from R2; value 4.7kΩ -> 1kΩ
- R10, R11, R12, R19, R20, R21, R26, R27, R36, R37, R38, R39, R9: value 4.7kΩ -> 68Ω
- R13: renamed from R6; value 4.7kΩ -> 1kΩ
- R14: renamed from R4; value 4.7kΩ -> 1kΩ
- R15: renamed from R16; value 4.7kΩ -> 1kΩ
- R2: renamed from R1; value 4.7kΩ -> 1kΩ
- R22: renamed from R17; value 4.7kΩ -> 1kΩ
- R23: renamed from R18; value 4.7kΩ -> 1kΩ
- R24, R25, R28, R29, R30, R31, R32, R33, R34, R35, R40, R7: value 4.7kΩ -> 1kΩ
- R3: renamed from R5; value 4.7kΩ -> 1kΩ
- R4: renamed from R3; value 4.7kΩ -> 1kΩ
- R5: renamed from R8; value 4.7kΩ -> 1kΩ
- moved Q20 287.7 mm to (-111.5, 148.1), turned to 0 degrees
- moved Q19 279.6 mm to (-111.5, 142.1), turned to 0 degrees
- moved Q18 273.6 mm to (-111.5, 136.1), turned to 0 degrees
- moved Q17 266.1 mm to (-111.5, 130.2), turned to 0 degrees
- moved Q16 260.0 mm to (-111.5, 124.2), turned to 0 degrees
- moved D18 255.5 mm to (-101.6, 59.1), turned to 0 degrees
- moved Q15 253.1 mm to (-111.5, 118.3), turned to 0 degrees
- moved D17 251.6 mm to (-101.6, 55.5), turned to 0 degrees
- moved Q14 246.6 mm to (-111.5, 112.3), turned to 0 degrees
- moved D20 245.8 mm to (-90.0, 147.2), turned to 0 degrees
- moved L16 242.7 mm to (-93.8, 120.5)
- moved D19 240.5 mm to (-90.0, 144.1), turned to 0 degrees
- moved Q13 240.4 mm to (-111.5, 106.3), turned to 0 degrees
- moved D14 238.2 mm to (-101.6, 52.0), turned to 0 degrees
- moved D16 236.9 mm to (-90.0, 51.7), turned to 0 degrees
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- renumbered D6 to D1
Connections:
- D12 pad 1: Net-(D12-K) -> +12v
- D12 pad 2: +12v -> Net-(D12-A)
- D13 pad 1: Net-(D13-K) -> +12v
- D13 pad 2: +12v -> Net-(D13-A)
- D14 pad 1: Net-(D14-K) -> +12v
- D14 pad 2: +12v -> Net-(D14-A)
- D17 pad 1: Net-(D17-K) -> +12v
- D17 pad 2: +12v -> Net-(D17-A)
- D18 pad 1: Net-(D18-K) -> +12v
- D18 pad 2: +12v -> Net-(D18-A)
- D5 pad 1: Net-(D5-K) -> +12v
- D5 pad 2: +12v -> Net-(D5-A)
- D7 pad 1: Net-(D7-K) -> +12v
- D7 pad 2: +12v -> Net-(D7-A)
- D8 pad 1: Net-(D8-K) -> +12v
- D8 pad 2: +12v -> Net-(D8-A)
- L1 pad 2: Net-(Q2-C) -> Net-(Q1-D)
- L10 pad 2: Net-(Q10-C) -> Net-(Q10-D)
- L11 pad 2: Net-(Q11-C) -> Net-(Q11-D)
- L12 pad 2: Net-(Q12-C) -> Net-(Q12-D)
- L13 pad 2: Net-(Q13-C) -> Net-(Q13-D)
- L3 pad 2: Net-(Q3-C) -> Net-(Q3-D)
- L4 pad 2: Net-(Q4-C) -> Net-(Q4-D)
- L5 pad 2: Net-(Q5-C) -> Net-(Q5-D)
- L6 pad 2: Net-(Q6-C) -> Net-(Q6-D)
- L7 pad 2: Net-(Q7-C) -> Net-(Q7-D)
- L8 pad 2: Net-(Q8-C) -> Net-(Q8-D)
- L9 pad 2: Net-(Q9-C) -> Net-(Q9-D)
- Q1 pad 1: Net-(Q1-B) -> Net-(Q1-G)
- Q1 pad 2: Net-(Q1-C) -> Net-(Q1-D)
- Q10 pad 1: Net-(Q10-B) -> Net-(Q10-G)
- Q10 pad 2: Net-(Q10-C) -> Net-(Q10-D)
- Q11 pad 1: Net-(Q11-B) -> Net-(Q11-G)
- Q11 pad 2: Net-(Q11-C) -> Net-(Q11-D)
- Q12 pad 1: Net-(Q12-B) -> Net-(Q12-G)
- Q12 pad 2: Net-(Q12-C) -> Net-(Q12-D)
- Q13 pad 1: Net-(Q13-B) -> Net-(Q13-G)
- Q13 pad 2: Net-(Q13-C) -> Net-(Q13-D)
- Q14 pad 1: Net-(Q14-B) -> Net-(Q14-G)
- Q15 pad 1: Net-(Q15-B) -> Net-(Q15-G)
- Q16 pad 1: Net-(Q16-B) -> Net-(Q16-G)
- Q17 pad 1: Net-(Q17-B) -> Net-(Q17-G)
- Q18 pad 1: Net-(Q18-B) -> Net-(Q18-G)
- Q19 pad 1: Net-(Q19-B) -> Net-(Q19-G)
- Q2 pad 1: Net-(Q2-B) -> Net-(Q2-G)
- Q2 pad 2: Net-(Q2-C) -> Net-(Q2-D)
- Q20 pad 1: Net-(Q20-B) -> Net-(Q20-G)
- Q3 pad 1: Net-(Q3-B) -> Net-(Q3-G)
- Q3 pad 2: Net-(Q3-C) -> Net-(Q3-D)
- Q4 pad 1: Net-(Q4-B) -> Net-(Q4-G)
- Q4 pad 2: Net-(Q4-C) -> Net-(Q4-D)
- Q5 pad 1: Net-(Q5-B) -> Net-(Q5-G)
- Q5 pad 2: Net-(Q5-C) -> Net-(Q5-D)
- Q6 pad 1: Net-(Q6-B) -> Net-(Q6-G)
- Q6 pad 2: Net-(Q6-C) -> Net-(Q6-D)
- Q7 pad 1: Net-(Q7-B) -> Net-(Q7-G)
- Q7 pad 2: Net-(Q7-C) -> Net-(Q7-D)
- Q8 pad 1: Net-(Q8-B) -> Net-(Q8-G)
- Q8 pad 2: Net-(Q8-C) -> Net-(Q8-D)
- Q9 pad 1: Net-(Q9-B) -> Net-(Q9-G)
- Q9 pad 2: Net-(Q9-C) -> Net-(Q9-D)
- R10 pad 1: Net-(R10-Pad1) -> Net-(Q2-D)
- R10 pad 2: Net-(Q4-B) -> Net-(D6-A)
- R11 pad 1: Net-(R11-Pad1) -> Net-(Q3-D)
- R11 pad 2: Net-(Q5-B) -> Net-(D7-A)
- R12 pad 1: Net-(R12-Pad1) -> Net-(Q4-D)
- R12 pad 2: Net-(Q6-B) -> Net-(D8-A)
- R19 pad 1: Net-(R19-Pad1) -> Net-(Q5-D)
- R19 pad 2: Net-(Q7-B) -> Net-(D12-A)
- R20 pad 1: Net-(R20-Pad1) -> Net-(Q6-D)
- R20 pad 2: Net-(Q8-B) -> Net-(D13-A)
- R21 pad 1: Net-(R21-Pad1) -> Net-(Q7-D)
- R21 pad 2: Net-(Q9-B) -> Net-(D14-A)
- R24 pad 1: Net-(R24-Pad1) -> Chassis_GND
- R24 pad 2: Net-(Q12-B) -> Net-(Q8-G)
- R25 pad 1: GND -> Chassis_GND
- R25 pad 2: Net-(R25-Pad2) -> Net-(Q9-G)
- R26 pad 1: GND -> Net-(Q8-D)
- R26 pad 2: Net-(R26-Pad2) -> Net-(D17-A)
- R27 pad 1: GND -> Net-(Q9-D)
- R27 pad 2: Net-(R27-Pad2) -> Net-(D18-A)
- R29 pad 1: Net-(R29-Pad1) -> GND
- R29 pad 2: Net-(Q13-B) -> Net-(R29-Pad2)
- R30 pad 1: Net-(R30-Pad1) -> GND
- R30 pad 2: Net-(Q14-B) -> Net-(R30-Pad2)
- R31 pad 1: Net-(R31-Pad1) -> GND
- R31 pad 2: Net-(Q15-B) -> Net-(R31-Pad2)
- R32 pad 1: Net-(R32-Pad1) -> Chassis_GND
- R32 pad 2: Net-(Q16-B) -> Net-(Q10-G)
- R33 pad 1: GND -> Chassis_GND
- R33 pad 2: Net-(R33-Pad2) -> Net-(Q11-G)
- R34 pad 1: GND -> Chassis_GND
- R34 pad 2: Net-(R34-Pad2) -> Net-(Q12-G)
- R35 pad 1: GND -> Chassis_GND
- R35 pad 2: Net-(R35-Pad2) -> Net-(Q13-G)
- R36 pad 1: GND -> Net-(Q10-D)
- R36 pad 2: Net-(R36-Pad2) -> Net-(D23-A)
- R37 pad 1: Net-(R37-Pad1) -> Net-(Q11-D)
- R37 pad 2: Net-(Q17-B) -> Net-(D24-A)
- R38 pad 1: Net-(R38-Pad1) -> Net-(Q12-D)
- R38 pad 2: Net-(Q18-B) -> Net-(D25-A)
- R39 pad 1: Net-(R39-Pad1) -> Net-(Q13-D)
- R39 pad 2: Net-(Q19-B) -> Net-(D26-A)
- R40 pad 1: Net-(R40-Pad1) -> GND
- R40 pad 2: Net-(Q20-B) -> Net-(R40-Pad2)
- R5 pad 1: Net-(R8-Pad1) -> Chassis_GND
- R5 pad 2: Net-(Q2-B) -> Net-(Q1-G)
- R7 pad 1: Net-(R7-Pad1) -> Chassis_GND
- R7 pad 2: Net-(Q1-B) -> Net-(Q3-G)
- R9 pad 1: Net-(R9-Pad1) -> Net-(Q1-D)
- R9 pad 2: Net-(Q3-B) -> Net-(D5-A)
- U1 pad 11: Net-(R10-Pad1) -> Net-(Q3-G)
- U1 pad 13: Net-(R7-Pad1) -> Net-(Q2-G)
- U1 pad 15: Net-(R8-Pad1) -> Net-(Q1-G)
- U1 pad 9: Net-(R11-Pad1) -> Net-(Q4-G)
- U2 pad 10: Net-(D10-K) -> Net-(D15-K)
- U2 pad 11: Net-(R22-Pad1) -> Net-(Q7-G)
- U2 pad 12: Net-(D12-K) -> Net-(D11-K)
- U2 pad 13: Net-(R9-Pad1) -> Net-(Q6-G)
- U2 pad 14: Net-(D1-K) (its old number) -> Net-(D10-K)
- U2 pad 15: Net-(R12-Pad1) -> Net-(Q5-G)
- U2 pad 16: Net-(D5-K) -> Net-(D9-K)
- U2 pad 9: Net-(R23-Pad1) -> Net-(Q8-G)
- U3 pad 10: Net-(D9-K) -> Net-(D22-K)
- U3 pad 11: Net-(R20-Pad1) -> Net-(Q12-G)
- U3 pad 12: Net-(D8-K) -> Net-(D21-K)
- U3 pad 13: Net-(R19-Pad1) -> Net-(Q11-G)
- U3 pad 14: Net-(D7-K) -> Net-(D20-K)
- U3 pad 15: Net-(R24-Pad1) -> Net-(Q9-G)
- U3 pad 16: Net-(D11-K) -> Net-(D16-K)
- U3 pad 4: Net-(R13-Pad2) (its old number) -> Net-(R29-Pad2)
- U3 pad 6: Net-(R14-Pad2) (its old number) -> Net-(R30-Pad2)
- U3 pad 8: Net-(R15-Pad2) (its old number) -> Net-(R31-Pad2)
- U3 pad 9: Net-(R21-Pad1) -> Net-(Q13-G)
- U4 pad 10: Net-(D16-K) -> Net-(D29-K)
- U4 pad 11: Net-(R31-Pad1) -> Net-(Q15-G)
- U4 pad 12: Net-(D15-K) -> Net-(D28-K)
- U4 pad 13: Net-(R30-Pad1) -> Net-(Q17-G)
- U4 pad 14: Net-(D14-K) -> Net-(D30-K)
- U4 pad 15: Net-(R29-Pad1) -> Net-(Q10-G)
- U4 pad 16: Net-(D13-K) -> Net-(D19-K)
- U4 pad 2: Net-(R25-Pad2) -> Net-(R28-Pad2)
- U4 pad 4: Net-(R26-Pad2) -> Net-(R43-Pad2)
- U4 pad 6: Net-(R27-Pad2) -> Net-(R41-Pad2)
- U4 pad 8: Net-(R28-Pad2) -> Net-(R42-Pad2)
- U4 pad 9: Net-(R32-Pad1) -> Net-(Q16-G)
- U5 pad 10: Net-(D20-K) -> Net-(D37-K)
- U5 pad 11: Net-(R39-Pad1) -> Net-(Q19-G)
- U5 pad 12: Net-(D19-K) -> Net-(D36-K)
- U5 pad 13: Net-(R38-Pad1) -> Net-(Q18-G)
- U5 pad 14: Net-(D18-K) -> Net-(D35-K)
- U5 pad 15: Net-(R37-Pad1) -> Net-(Q14-G)
- U5 pad 16: Net-(D17-K) -> Net-(D27-K)
- U5 pad 2: Net-(R33-Pad2) -> Net-(R40-Pad2)
- U5 pad 4: Net-(R34-Pad2) -> Net-(R52-Pad2)
- U5 pad 6: Net-(R35-Pad2) -> Net-(R53-Pad2)
- U5 pad 8: Net-(R36-Pad2) -> Net-(R54-Pad2)
- U5 pad 9: Net-(R40-Pad1) -> Net-(Q20-G)
Routing:
- net +12v: track 416.3 -> 0.00 mm
- net Net-(R8-Pad1): track 31.0 -> 0.00 mm
- net Net-(R40-Pad1): track 28.3 -> 0.00 mm
- net Net-(R7-Pad1): track 28.1 -> 0.00 mm
- net Net-(D20-K): track 26.6 -> 0.00 mm
- net Net-(R39-Pad1): track 26.4 -> 0.00 mm
- net Net-(D3-K): track 25.2 -> 0.00 mm
- net Net-(R10-Pad1): track 25.0 -> 0.00 mm
- net Net-(Q20-B): track 24.9 -> 0.00 mm
- net Net-(D19-K): track 24.1 -> 0.00 mm
- net Net-(R38-Pad1): track 23.5 -> 0.00 mm
- net Net-(Q18-B): track 22.9 -> 0.00 mm
- net Net-(R32-Pad1): track 22.2 -> 0.00 mm
- net Net-(D4-K): track 22.0 -> 0.00 mm
- net Net-(D18-K): track 21.5 -> 0.00 mm
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
Commit message: replaced footprints on breakout to match new components
Parts:
- Q1, Q10, Q11, Q12, Q13, Q14, Q15, Q16, Q17, Q18, Q19, Q20, Q7, Q8, Q9: footprint Package_TO_SOT_THT:TO-220-3_Vertical -> Package_TO_SOT_THT:TO-220-3_Horizontal_TabUp
- Q2, Q3, Q4, Q5, Q6: footprint Package_TO_SOT_THT:TO-220-3_Vertical -> Package_TO_SOT_THT:TO-220-3_Horizontal_TabUp; moved to B.Cu
- R10, R11, R12, R19, R20, R21, R26, R27, R36, R37, R38, R39, R48, R49, R50, R51, R58, R59, R60, R9: value 68Ω -> 1kΩ-P; footprint Resistor_SMD:R_0805_2012Metric_Pad1.20x1.40mm_HandSolder -> Resistor_SMD:R_1206_3216Metric_Pad1.30x1.75mm_HandSolder
- moved J3 274.3 mm to (175.9, 127.0), turned to 90 degrees
- moved Q6 235.4 mm to (120.7, 101.6), turned to 180 degrees
- moved Q5 224.8 mm to (104.1, 120.0)
- moved Q4 215.4 mm to (97.8, 101.6), turned to 180 degrees
- moved Q3 207.0 mm to (81.3, 120.0)
- moved R16 198.9 mm to (105.1, 116.8), turned to 180 degrees
- moved Q2 196.7 mm to (74.9, 101.6), turned to 180 degrees
- moved R8 185.9 mm to (94.0, 104.8)
- moved R7 178.6 mm to (82.3, 116.8), turned to 180 degrees
- moved J2 24.1 mm to (48.9, 127.0), turned to -90 degrees
- moved R6 21.6 mm to (70.2, 104.8), turned to 0 degrees
- moved R5 9.30 mm to (59.3, 116.8), turned to 180 degrees
- moved D3 5.51 mm to (69.2, 132.7)
- moved Q1 2.54 mm to (58.4, 120.0)
Connections:
- J3 pad 1: +12v -> Chassis_GND
- J3 pad 2: Chassis_GND -> +12v

Commit message: finished rev B pcb for solenoid breakout
Parts:
- added REF**: 6-32 Mount, OF Footprints:6-32 Mount, F.Cu at (48.3, 57.1)
- added REF**: 6-32 Mount, OF Footprints:6-32 Mount, F.Cu at (48.3, 151.8)
- added REF**: 6-32 Mount, OF Footprints:6-32 Mount, F.Cu at (184.8, 151.8)
- added REF**: 6-32 Mount, OF Footprints:6-32 Mount, F.Cu at (184.8, 57.1)
- L15: moved to F.Cu
- Q10, Q11, Q12, Q13, Q14, Q15, Q16, Q17, Q18, Q19, Q20, Q7, Q8, Q9: moved to B.Cu
- moved D40 304.4 mm to (185.7, 79.4), turned to 180 degrees
- moved D33 300.6 mm to (181.6, 65.2), turned to -90 degrees
- moved D38 299.4 mm to (186.3, 90.8), turned to 180 degrees
- moved Q20 298.7 mm to (177.8, 73.9), turned to 180 degrees
- moved D39 293.4 mm to (185.8, 117.5), turned to 180 degrees
- moved D31 292.5 mm to (185.7, 103.5), turned to 180 degrees
- moved D32 291.6 mm to (173.4, 65.2), turned to -90 degrees
- moved D34 286.3 mm to (165.1, 65.2), turned to -90 degrees
- moved Q19 285.6 mm to (172.7, 114.2)
- moved Q18 283.5 mm to (165.1, 73.9), turned to 180 degrees
- moved L16 276.6 mm to (177.2, 64.8)
- moved Q14 271.5 mm to (160.0, 114.2)
- moved D23 270.3 mm to (156.8, 65.2), turned to -90 degrees
- moved Q16 268.7 mm to (152.4, 73.9), turned to 180 degrees
- moved D37 266.0 mm to (178.4, 121.3), turned to 90 degrees
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Routing:
- net +12v: track 0.00 -> 411.9 mm
- net Net-(Q18-G): track 0.00 -> 102.1 mm
- net Net-(Q20-G): track 0.00 -> 101.1 mm
- net Net-(Q16-G): track 0.00 -> 96.1 mm
- net Net-(Q17-G): track 0.00 -> 91.7 mm
- net Net-(Q2-G): track 0.00 -> 85.5 mm
- net Net-(Q13-G): track 0.00 -> 85.0 mm
- net Net-(Q11-G): track 0.00 -> 78.3 mm
- net Net-(Q8-G): track 0.00 -> 74.8 mm
- net Net-(Q4-G): track 0.00 -> 73.5 mm
- net Net-(Q6-G): track 0.00 -> 72.5 mm
- net Net-(Q9-D): track 0.00 -> 63.7 mm
- net Net-(Q15-D): track 0.00 -> 62.4 mm
- net Net-(Q10-D): track 0.00 -> 59.9 mm
- net Net-(Q19-G): track 0.00 -> 59.3 mm
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Other:
- board size 135.9 x 67.9 mm -> 144.1 x 102.2 mm
- board text added: "Solenoid Breakout Board Rev. B Designed By: Owen Fujii 04/02/2025"
- board text removed: "Solenoid Breakout Board Rev. A Designed By: Owen Fujii 03/10/2025"
