File: Solenoid Breakout Board/Solenoid Breakout Board.kicad_sch (KiCad schematic)
At the start: 106 parts, among them J1 Solenoid In, Q13 STN851-A, Q14 STN851-A, Q15 STN851-A, Q16 STN851-A, Q17 STN851-A, Q18 STN851-A, Q19 STN851-A, Q20 STN851-A, Q21 STN851-A, Q22 STN851-A, Q23 STN851-A, Q24 STN851-A, Q25 STN851-A, Q26 STN851-A, Q27 STN851-A, Q28 STN851-A, Q29 STN851-A, Q30 STN851-A, Q31 STN851-A, Q32 STN851-A, U11 LTV-247, U12 LTV-247, U13 LTV-247, U14 LTV-247, U15 LTV-247

Commit message: finished rev A pcb for breakout:
Parts:
- added J2: Pwr IN, Connector_PinHeader_2.54mm:PinHeader_1x02_P2.54mm_Vertical, symbol Owen's Symbols:Header_1x2
Connections:
- net +12v: now also J2.1
- net Chassis_GND: now also J2.2
Changed lines of the file:
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@@
 	(wire
 		(pts
+			(xy 22.86 151.13) (xy 22.86 153.67)
+		)
+		(stroke
+			(width 0)
+			(type default)
+		)
+	)
+	(wire
+		(pts
+			(xy 20.32 151.13) (xy 22.86 151.13)
+		)
+		(stroke
+			(width 0)
+			(type default)
+		)
+	)
+	(wire
+		(pts
 			(xy 20.32 102.87) (xy 24.13 102.87)
 		)
@@
 	(wire
 		(pts
+			(xy 22.86 148.59) (xy 22.86 147.32)
+		)
+		(stroke
+			(width 0)
+			(type default)
+		)
+	)
+	(wire
+		(pts
 			(xy 95.25 158.75) (xy 95.25 161.29)
 		)
@@
 	(wire
 		(pts
+			(xy 20.32 148.59) (xy 22.86 148.59)
+		)
+		(stroke
+			(width 0)
+			(type default)
+		)
+	)
+	(wire
+		(pts
 			(xy 68.58 53.34) (xy 76.2 53.34)
 		)
@@
 	)
 	(symbol
+		(lib_id "Owen's Symbols:Header_1x2")
+		(at 20.32 148.59 0)
+		(unit 1)
+		(exclude_from_sim no)
+		(in_bom yes)
+		(on_board yes)
+		(dnp no)
+		(fields_autoplaced yes)
+		(property "Reference" "J2"
+			(at 16.51 140.97 0)
+			(effects
+				(font
+					(size 1.27 1.27)
+				)
+			)
+		)
+		(property "Value" "Pwr IN"
+			(at 16.51 143.51 0)
+			(effects
+				(font
+					(size 1.27 1.27)
+				)
+			)
+		)
+		(property "Footprint" "Connector_PinHeader_2.54mm:PinHeader_1x02_P2.54mm_Vertical"
+			(at 16.51 144.78 0)
+			(effects
+				(font
+					(size 1.27 1.27)
+				)
+				(hide yes)
+			)
+		)
+		(property "Datasheet" ""
+			(at 16.51 144.78 0)
+			(effects
+				(font
+					(size 1.27 1.27)
+				)
+				(hide yes)
+			)
+		)
+		(property "Description" ""
+			(at 20.32 148.59 0)
+			(effects
+				(font
+					(size 1.27 1.27)
+				)
+				(hide yes)
+			)
+		)
+		(pin "2"
+		)
+		(pin "1"
+		)
+		(instances
+			(project ""
+				(path "/2b4cb468-ebc7-4952-9328-7c324ac62f95"
+					(reference "J2")
+					(unit 1)
+				)
+			)
+		)
+	)
+	(symbol
 		(lib_id "Custom Symbols:Resistor_Mod")
 		(at 171.45 34.29 0)
@@
 	)
 	(symbol
+		(lib_id "Custom Power:Chassis_GND")
+		(at 22.86 153.67 0)
+		(unit 1)
+		(exclude_from_sim no)
+		(in_bom no)
+		(on_board no)
+		(dnp no)
+		(fields_autoplaced yes)
+		(property "Reference" "#PWR062"
+			(at 22.86 152.4 0)
+			(effects
+				(font
+					(size 1.27 1.27)
+				)
+				(hide yes)
+			)
+		)
+		(property "Value" "Chassis_GND"
+			(at 22.86 152.4 0)
+			(effects
+				(font
+					(size 1.27 1.27)
+				)
+				(hide yes)
+			)
+		)
+		(property "Footprint" ""
+			(at 22.86 152.4 0)
+			(effects
+				(font
+					(size 1.27 1.27)
+				)
+				(hide yes)
+			)
+		)
+		(property "Datasheet" ""
+			(at 22.86 152.4 0)
+			(effects
+				(font
+					(size 1.27 1.27)
+				)
+				(hide yes)
+			)
+		)
+		(property "Description" ""
+			(at 22.86 153.67 0)
+			(effects
+				(font
+					(size 1.27 1.27)
+				)
+				(hide yes)
+			)
+		)
+		(pin "1"
+		)
+		(instances
+			(project "Solenoid Breakout Board"
+				(path "/2b4cb468-ebc7-4952-9328-7c324ac62f95"
+					(reference "#PWR062")
+					(unit 1)
+				)
+			)
+		)
+	)
+	(symbol
 		(lib_id "Device:Q_NPN_BCE")
 		(at 182.88 66.04 0)
@@
 					(unit 1)
 				)
+			)
+		)
+	)
+	(symbol
+		(lib_id "Custom Power:+12v")
+		(at 22.86 146.05 0)
+		(unit 1)
+		(exclude_from_sim no)
+		(in_bom no)
+		(on_board no)
+		(dnp no)
+		(fields_autoplaced yes)
+		(property "Reference" "#PWR063"
+			(at 27.5844 142.3416 0)
+			(effects
+				(font
+					(size 1.27 1.27)
+				)
+				(hide yes)
+			)
+		)
+		(property "Value" "+12v"
+			(at 22.86 140.97 0)
+			(effects
+				(font
+					(size 1.27 1.27)
+				)
+			)
+		)
+		(property "Footprint" ""
+			(at 22.86 142.24 0)
+			(effects
+				(font
+					(size 1.27 1.27)
+				)
+				(hide yes)
+			)
+		)
+		(property "Datasheet" ""
+			(at 22.86 142.24 0)
+			(effects
+				(font
+					(size 1.27 1.27)
+				)
+				(hide yes)
+			)
+		)
+		(property "Description" ""
+			(at 22.86 146.05 0)
+			(effects
+				(font
+					(size 1.27 1.27)
+				)
+				(hide yes)
+			)
+		)
+		(pin "~"
+		)
+		(instances
+			(project "Solenoid Breakout Board"
+				(path "/2b4cb468-ebc7-4952-9328-7c324ac62f95"
+					(reference "#PWR063")
+					(unit 1)
+				)

Commit message: currently revising solenoid breakout to match new design
Parts:
- removed D23, D24, D25, D26, D27, D29, D30, D31, D32, D33, D34, D35, D36, D37, D38, D39, D40, D41, D42: LED, LED_SMD:LED_0805_2012Metric_Pad1.15x1.40mm_HandSolder, symbol Device:LED
- removed L13, L14, L15, L16, L17, L19, L20, L21, L22, L23, L24, L25, L26, L27, L28, L29, L30, L31, L32: Solenoid, Connector_PinHeader_2.54mm:PinHeader_1x02_P2.54mm_Vertical, symbol Device:L
- removed Q13, Q14, Q15, Q16, Q17, Q18, Q19, Q20, Q21, Q22, Q23, Q24, Q25, Q26, Q27, Q28, Q29, Q30, Q31, Q32: STN851-A, Package_TO_SOT_SMD:SOT-223-3_TabPin2, symbol Device:Q_NPN_BCE
- removed R100, R101, R106, R107, R108, R109, R76, R77, R78, R79, R80, R88, R89, R90, R91, R92, R93, R98, R99: 4.7kΩ, Resistor_SMD:R_0805_2012Metric_Pad1.20x1.40mm_HandSolder, symbol Custom Symbols:Resistor_Mod
- added D10, D12, D14, D16, D8, D?: 1N4148, Diode_THT:D_DO-35_SOD27_P7.62mm_Horizontal, symbol Diode:1N4148
- added D11, D13, D15, D7, D9: LED, LED_SMD:LED_0805_2012Metric_Pad1.15x1.40mm_HandSolder, symbol Device:LED
- added J3: Pwr OUT, Connector_PinHeader_2.54mm:PinHeader_1x02_P2.54mm_Vertical, symbol Owen's Symbols:Header_1x2
- added L3, L4, L5, L6, L7: Solenoid, Connector_PinHeader_2.54mm:PinHeader_1x02_P2.54mm_Vertical, symbol Device:L
- added Q1, Q2, Q3, Q4, Q5, Q?: IRF540N, Package_TO_SOT_THT:TO-220-3_Vertical, symbol Transistor_FET:IRF540N
- added R10, R12, R20, R22, R24, R?: 68Ω, symbol OF symbols:Resistor_Mod
- added R11, R19, R21, R23, R9: 1kΩ, Resistor_SMD:R_0805_2012Metric_Pad1.20x1.40mm_HandSolder, symbol Custom Symbols:Resistor_Mod
- R1: renamed from R74; value 4.7kΩ -> 1kΩ
- R13: renamed from R82; value 4.7kΩ -> 1kΩ
- R14: renamed from R83; value 4.7kΩ -> 1kΩ
- R15: renamed from R84; value 4.7kΩ -> 1kΩ
- R16: renamed from R85; value 4.7kΩ -> 1kΩ
- R17: renamed from R86; value 4.7kΩ -> 1kΩ
- R18: renamed from R87; value 4.7kΩ -> 1kΩ
- R2: renamed from R75; value 4.7kΩ -> 1kΩ
- R25: renamed from R94; value 4.7kΩ -> 1kΩ
- R26: renamed from R95; value 4.7kΩ -> 1kΩ
- R27: renamed from R96; value 4.7kΩ -> 1kΩ
- R28: renamed from R97; value 4.7kΩ -> 1kΩ
- R3: renamed from R70; value 4.7kΩ -> 1kΩ
- R33: renamed from R102; value 4.7kΩ -> 1kΩ
- R34: renamed from R103; value 4.7kΩ -> 1kΩ
- R35: renamed from R104; value 4.7kΩ -> 1kΩ
- R36: renamed from R105; value 4.7kΩ -> 1kΩ
- R4: renamed from R71; value 4.7kΩ -> 1kΩ
- R5: renamed from R72; value 4.7kΩ -> 1kΩ
- R6: renamed from R73; value 4.7kΩ -> 1kΩ
- R8: renamed from R81; value 4.7kΩ -> 1kΩ
- renumbered D28 to D6, L18 to L2, U12 to U1, U11 to U1, U11 to U2, U13 to U2, U12 to U3, U13 to U3, U14 to U4, U15 to U5
Connections:
- net +12v: now also D10.1 (K), D11.2 (A), D12.1 (K), D13.2 (A), D14.1 (K), D15.2 (A), D16.1 (K), D7.2 (A), D8.1 (K), D9.2 (A), D?.1 (K), J3.1, L3.1, L4.1, L5.1, L6.1, L7.1
- net Chassis_GND: now also R8.1, J3.2, Q1.3 (S), Q2.3 (S), Q3.3 (S), Q4.3 (S), Q5.3 (S), Q?.3 (S), R11.1, R19.1, R21.1, R23.1, R9.1
- net at U2.13: now also Q5.1 (G), R23.2
- net at U2.14: now also D15.1 (K)
- net at U1.11: now also Q2.1 (G), R11.2
- net at U2.15: now also Q4.1 (G), R21.2
- net at U2.16: now also D13.1 (K)
- net at U1.10: now also D11.1 (K)
- net at U1.15: now also R8.2, Q?.1 (G); no longer R8.1
- net at U1.9: now also Q3.1 (G), R19.2
- net at U1.14: now also D7.1 (K)
- net at L2.2: now also Q?.2 (D), R?.1
- net at U1.12: now also D9.1 (K)
- net at U1.13: now also Q1.1 (G), R9.2
- new net: D12.2 (A), R20.2
- new net: L6.2, Q4.2 (D), R22.1
- new net: L7.2, Q5.2 (D), R24.1
- new net: D14.2 (A), R22.2
- new net: D10.2 (A), R12.2
- new net: L3.2, Q1.2 (D), R10.1
- new net: D8.2 (A), R10.2
- new net: L4.2, Q2.2 (D), R12.1
- new net: L5.2, Q3.2 (D), R20.1
- new net: D16.2 (A), R24.2
- new net: D?.2 (A), R?.2
Other:
- moved on the sheet: D6, L2, R1, R13, R14, R15, R16, R17, R18, R2, R25, R26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

Commit message: revised schematic for breakout updating PCB to match
Parts:
- removed R13, R14, R15, R25, R26, R27, R28, R33, R34, R35, R36: 1kΩ, Resistor_SMD:R_0805_2012Metric_Pad1.20x1.40mm_HandSolder, symbol Owen's Symbols:Resistor_Mod
- removed unit 3 of U3
- removed unit 4 of U3
- removed unit 2 of U3
- removed U4, U5: LTV-247, Package_SO:SOP-16_4.4x10.4mm_P1.27mm, symbol Isolator:LTV-247
- added D11, D15, D16: LED, LED_SMD:LED_0805_2012Metric_Pad1.15x1.40mm_HandSolder, symbol Device:LED
- added D14, D17, D18: 1N4148, LED_SMD:LED_0805_2012Metric_Pad1.15x1.40mm_HandSolder, symbol Diode:1N4148
- added L7, L8, L9: Solenoid, OF Footprints:Small Expanded TH, symbol Device:L
- added Q7, Q8, Q9: IRF540N, Package_TO_SOT_THT:TO-220-3_Vertical, symbol Transistor_FET:IRF540N
- added R18, R24, R25: 1kΩ, Resistor_SMD:R_0805_2012Metric_Pad1.20x1.40mm_HandSolder, symbol Custom Symbols:Resistor_Mod
- added R21, R26, R27: 68Ω, Resistor_SMD:R_0805_2012Metric_Pad1.20x1.40mm_HandSolder, symbol OF symbols:Resistor_Mod
- D12: renamed from D14; footprint Diode_THT:D_DO-35_SOD27_P7.62mm_Horizontal -> LED_SMD:LED_0805_2012Metric_Pad1.15x1.40mm_HandSolder
- D13: renamed from D16; footprint Diode_THT:D_DO-35_SOD27_P7.62mm_Horizontal -> LED_SMD:LED_0805_2012Metric_Pad1.15x1.40mm_HandSolder
- D5: renamed from D?; footprint Diode_THT:D_DO-35_SOD27_P7.62mm_Horizontal -> LED_SMD:LED_0805_2012Metric_Pad1.15x1.40mm_HandSolder
- D6: renamed from D8; footprint Diode_THT:D_DO-35_SOD27_P7.62mm_Horizontal -> LED_SMD:LED_0805_2012Metric_Pad1.15x1.40mm_HandSolder
- D7: renamed from D10; footprint Diode_THT:D_DO-35_SOD27_P7.62mm_Horizontal -> LED_SMD:LED_0805_2012Metric_Pad1.15x1.40mm_HandSolder
- D8: renamed from D12; footprint Diode_THT:D_DO-35_SOD27_P7.62mm_Horizontal -> LED_SMD:LED_0805_2012Metric_Pad1.15x1.40mm_HandSolder
- J2, J3: footprint Connector_PinHeader_2.54mm:PinHeader_1x02_P2.54mm_Vertical -> OF Footprints:Two_Pin_Screw_Terminal
- L1: renamed from L2; footprint Connector_PinHeader_2.54mm:PinHeader_1x02_P2.54mm_Vertical -> OF Footprints:Small Expanded TH
- L2: renamed from L3; footprint Connector_PinHeader_2.54mm:PinHeader_1x02_P2.54mm_Vertical -> OF Footprints:Small Expanded TH
- L3: renamed from L4; footprint Connector_PinHeader_2.54mm:PinHeader_1x02_P2.54mm_Vertical -> OF Footprints:Small Expanded TH
- L4: renamed from L5; footprint Connector_PinHeader_2.54mm:PinHeader_1x02_P2.54mm_Vertical -> OF Footprints:Small Expanded TH
- L5: renamed from L6; footprint Connector_PinHeader_2.54mm:PinHeader_1x02_P2.54mm_Vertical -> OF Footprints:Small Expanded TH
- L6: renamed from L7; footprint Connector_PinHeader_2.54mm:PinHeader_1x02_P2.54mm_Vertical -> OF Footprints:Small Expanded TH
- R10: footprint (none) -> Resistor_SMD:R_0805_2012Metric_Pad1.20x1.40mm_HandSolder
- R11: renamed from R12; footprint (none) -> Resistor_SMD:R_0805_2012Metric_Pad1.20x1.40mm_HandSolder
- R12: renamed from R20; footprint (none) -> Resistor_SMD:R_0805_2012Metric_Pad1.20x1.40mm_HandSolder
- R19: renamed from R22; footprint (none) -> Resistor_SMD:R_0805_2012Metric_Pad1.20x1.40mm_HandSolder
- R20: renamed from R24; footprint (none) -> Resistor_SMD:R_0805_2012Metric_Pad1.20x1.40mm_HandSolder
- R9: renamed from R?; footprint (none) -> Resistor_SMD:R_0805_2012Metric_Pad1.20x1.40mm_HandSolder
- gave numbers to parts that had none: 1
- renumbered D6 to D1, D15 to D10, D7 to D2, D9 to D3, D11 to D4, D13 to D9, Q1 to Q2, Q2 to Q3, Q3 to Q4, Q4 to Q5, Q5 to Q6, R2 to R1, R6 to R13, R4 to R14, R16 to R15, R21 to R16, R23 to R17, R1 to R2, R17 to R22, R18 to R23, R5 to R3, R3 to R4, R8 to R5, R9 to R6, R11 to R7, R19 to R8
Connections:
- net +12v: now also D11.2 (A), D14.1 (K), D15.2 (A), D16.2 (A), D17.1 (K), D18.1 (K), L7.1, L8.1, L9.1
- net Chassis_GND: now also Q7.3 (S), Q8.3 (S), Q9.3 (S), R18.1, R24.1, R25.1
- net at U2.10: now also D15.1 (K)
- net at U2.9: now also Q8.1 (G), R24.2
- net at U2.11: now also Q7.1 (G), R18.2
- net at U2.12: now also D11.1 (K)
- net at U3.15: now also Q9.1 (G), R25.2
- net at U3.16: now also D16.1 (K)
- new net: L8.2, Q8.2 (D), R26.1
- new net: L9.2, Q9.2 (D), R27.1
- new net: D18.2 (A), R27.2
- new net: D17.2 (A), R26.2
- new net: L7.2, Q7.2 (D), R21.1
- new net: D14.2 (A), R21.2
Other:
- added sheet Solenoids Extended (SolenoidsEx.kicad_sch)
- moved on the sheet: R15, R22, R23, U2C, U2D, U3A
