File: Motherboard Sch/Eslave Sch.kicad_sch (KiCad schematic)
At the start: 14 parts, among them J3 E SLAVE ISCP, J4 E Slave Out, J5 Solenoid In, SW3 E-slave Reset, U2 PIC16F1789

Commit message: renamed Midi bass sch to Motherboard Sch
Parts:
- D10: value E Active -> Fret Active
- D9: value E Status -> Fret Status
- J3: value E SLAVE ISCP -> FRET SLAVE ISCP
- J4: value E Slave Out -> Fret Out
- SW3: value E-slave Reset -> Fret Slave Reset
- TP5: value E CLKOUT -> FRET CLKOUT
Other:
- moved on the sheet: D10, R18
Changed lines of the file:
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@@
 	(wire
 		(pts
-			(xy 166.37 104.14) (xy 223.52 104.14)
+			(xy 166.37 104.14) (xy 227.33 104.14)
 		)
 		(stroke
@@
 	(wire
 		(pts
-			(xy 223.52 104.14) (xy 223.52 106.68)
+			(xy 227.33 104.14) (xy 227.33 106.68)
 		)
 		(stroke
@@
 	(wire
 		(pts
-			(xy 223.52 114.3) (xy 223.52 116.84)
+			(xy 227.33 114.3) (xy 227.33 116.84)
 		)
 		(stroke
@@
 			)
 		)
-		(property "Value" "E CLKOUT"
+		(property "Value" "FRET CLKOUT"
 			(at 168.91 28.4479 0)
 			(effects
@@
 	(symbol
 		(lib_id "Device:LED")
-		(at 223.52 120.65 90)
+		(at 227.33 120.65 90)
 		(unit 1)
 		(exclude_from_sim no)
@@
 		(fields_autoplaced yes)
 		(property "Reference" "D10"
-			(at 227.33 120.9674 90)
+			(at 231.14 120.9674 90)
 			(effects
 				(font
@@
 			)
 		)
-		(property "Value" "E Active"
-			(at 227.33 123.5074 90)
+		(property "Value" "Fret Active"
+			(at 231.14 123.5074 90)
 			(effects
 				(font
@@
 		)
 		(property "Footprint" "Diode_SMD:D_0805_2012Metric_Pad1.15x1.40mm_HandSolder"
-			(at 223.52 120.65 0)
+			(at 227.33 120.65 0)
 			(effects
 				(font
@@
 		)
 		(property "Datasheet" "~"
-			(at 223.52 120.65 0)
+			(at 227.33 120.65 0)
 			(effects
 				(font
@@
 		)
 		(property "Description" "Light emitting diode"
-			(at 223.52 120.65 0)
+			(at 227.33 120.65 0)
 			(effects
 				(font
@@
 	(symbol
 		(lib_id "Custom Power:GND")
-		(at 223.52 124.46 0)
+		(at 227.33 124.46 0)
 		(unit 1)
 		(exclude_from_sim no)
@@
 		(fields_autoplaced yes)
 		(property "Reference" "#PWR032"
-			(at 223.52 123.19 0)
+			(at 227.33 123.19 0)
 			(effects
 				(font
@@
 		)
 		(property "Value" "GND"
-			(at 223.52 123.19 0)
+			(at 227.33 123.19 0)
 			(effects
 				(font
@@
 		)
 		(property "Footprint" ""
-			(at 223.52 123.19 0)
+			(at 227.33 123.19 0)
 			(effects
 				(font
@@
 		)
 		(property "Datasheet" ""
-			(at 223.52 123.19 0)
+			(at 227.33 123.19 0)
 			(effects
 				(font
@@
 		)
 		(property "Description" ""
-			(at 223.52 124.46 0)
+			(at 227.33 124.46 0)
 			(effects
 				(font
@@
 			)
 		)
-		(property "Value" "E Slave Out"
+		(property "Value" "Fret Out"
 			(at 201.93 41.91 0)
 			(effects
@@
 			)
 		)
-		(property "Value" "E SLAVE ISCP"
+		(property "Value" "FRET SLAVE ISCP"
 			(at 25.4 46.99 0)
 			(effects
@@
 			)
 		)
-		(property "Value" "E-slave Reset"
+		(property "Value" "Fret Slave Reset"
 			(at 49.53 125.73 0)
 			(effects
@@
 	(symbol
 		(lib_id "Owen's Symbols:Resistor_Mod")
-		(at 223.52 110.49 90)
+		(at 227.33 110.49 90)
 		(unit 1)
 		(exclude_from_sim no)
@@
 		(fields_autoplaced yes)
 		(property "Reference" "R18"
-			(at 226.06 109.2199 90)
+			(at 229.87 109.2199 90)
 			(effects
 				(font
@@
 		)
 		(property "Value" "330Ω"
-			(at 226.06 111.7599 90)
+			(at 229.87 111.7599 90)
 			(effects
 				(font
@@
 		)
 		(property "Footprint" "Resistor_SMD:R_0805_2012Metric_Pad1.20x1.40mm_HandSolder"
-			(at 220.98 111.76 0)
+			(at 224.79 111.76 0)
 			(effects
 				(font
@@
 		)
 		(property "Datasheet" ""
-			(at 220.98 111.76 0)
+			(at 224.79 111.76 0)
 			(effects
 				(font
@@
 		)
 		(property "Description" ""
-			(at 223.52 110.49 0)
+			(at 227.33 110.49 0)
 			(effects
 				(font
@@
 			)
 		)
-		(property "Value" "E Status"
+		(property "Value" "Fret Status"
 			(at 213.36 126.0474 90)
 			(effects
