File: IR_MIDI/Midi_IR_Rx/Rx/Rx.kicad_sch (KiCad schematic)
At the start: 41 parts, among them J2 DIN-5, Q1 BPX38, Q2 2N3904, Q3 2N3904, Q4 2N3904, Q5 2N3904, Q6 2N3904, U1 4046, U2 SY21222

Commit message: updating for merge
Parts:
- removed C8, C9: 10µF, symbol Device:C_Polarized_Small_US
- removed D1: D_Schottky, symbol Device:D_Schottky
- removed L1: 6.8µH, symbol Device:L
- removed R19: 200KΩ, symbol Device:R_Small_US
- removed R20: 5.1KΩ, symbol Device:R_Small_US
- removed U2: SY21222, Package_TO_SOT_SMD:SOT-23-6, symbol Regulator_Switching:TLV61070ADBV
- J1: value ~ -> Power In
Connections:
- net at J1.1: now also J2.4, R1.2, R15.1, R17.1, R18.1, R5.2, R6.2, R8.2, R9.2, U1.16 (VDD)
- no-connect marks 7 -> 6
Other:
- moved on the sheet: C1, C2, C3, C4, C5, C6, C7, J1, J2, Q1, Q2, Q3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
